Commit message: working on urdf

File: urdf/minibot.urdf (robot description, URDF)
Before this commit: robot Minibot, 25 links, 24 joints
Links:
- link MP_ARM_HIGH_L: geometry collision mesh filename=package://minibot_description/meshes/upper_arm_low.stl scale=1 1 1; visual mesh filename=package://minibot_description/meshes/upper_arm_high.stl scale=1 1 1
- link MP_ARM_HIGH_R: geometry collision mesh filename=package://minibot_description/meshes/upper_arm_high.stl scale=1 1 1; visual mesh filename=package://minibot_description/meshes/upper_arm_high.stl scale=1 1 1
- link MP_BODY: geometry collision mesh filename=package://minibot_description/meshes/torso_low.stl scale=1 1 1; visual mesh filename=package://minibot_description/meshes/torso_high.stl scale=1 1 1
- link MP_SHOULDER_L: geometry collision mesh filename=package://minibot_description/meshes/shoulder_con_low.stl scale=1 1 1; visual mesh filename=package://minibot_description/meshes/shoulder_con_high.stl scale=1 1 1
- link MP_SHOULDER_R: geometry collision mesh filename=package://minibot_description/meshes/shoulder_con_low.stl scale=1 1 1; visual mesh filename=package://minibot_description/meshes/shoulder_con_high.stl scale=1 1 1
Joints:
- joint RShoulderRoll: origin xyz=0.016 0 0.02165 rpy=-1.5707963 1.5707963 0 -> xyz=0 0 0.029194 rpy=-1.5707963 1.5707963 0
- joint j_back_l: limit lower=-2.6179939 upper=2.6179939 effort=2.8 velocity=5.6548668 -> (none); origin xyz=0 0.06035 0 rpy=-1.5707963 0 0 -> xyz=0 0.08134 0 rpy=-1.5707963 0 0
- joint j_back_r: limit lower=-2.6179939 upper=2.6179939 effort=2.8 velocity=5.6548668 -> (none); origin xyz=0 -0.06035 0 rpy=1.5707963 0 0 -> xyz=0 -0.08134 0 rpy=1.5707963 0 0

Commit message: further work on urdf. visually now finished, but still problems with collision model

File: urdf/minibot.urdf (robot description, URDF)
Before this commit: robot Minibot, 25 links, 24 joints
Links:
- link MP_ANKLE1_L: geometry collision mesh filename=package://minibot_description/meshes/ankle_roll_low.stl scale=1 1 1; visual mesh filename=package://minibot_description/meshes/ankle_roll_high.stl scale=1 1 1
- link MP_ANKLE1_R: geometry collision mesh filename=package://minibot_description/meshes/ankle_roll_low.stl scale=1 1 1; visual mesh filename=package://minibot_description/meshes/ankle_roll_high.stl scale=1 1 1
- link MP_ANKLE2_L: geometry collision mesh filename=package://minibot_description/meshes/foot_low.stl scale=1 1 1; visual mesh filename=package://minibot_description/meshes/foot_high.stl scale=1 1 1
- link MP_ANKLE2_R: geometry collision mesh filename=package://minibot_description/meshes/foot_low.stl scale=1 1 1; visual mesh filename=package://minibot_description/meshes/foot_high.stl scale=1 1 1
- link MP_ARM_LOW_L: geometry collision mesh filename=package://minibot_description/meshes/lower_arm_low.stl scale=1 1 1; visual mesh filename=package://minibot_description/meshes/lower_arm_high.stl scale=1 1 1
- link MP_ARM_LOW_R: geometry collision mesh filename=package://minibot_description/meshes/lower_arm_low.stl scale=1 1 1; visual mesh filename=package://minibot_description/meshes/lower_arm_high.stl scale=1 1 1
- link MP_HEAD: geometry collision mesh filename=package://minibot_description/meshes/head_upper_low.stl scale=1 1 1; visual mesh filename=package://minibot_description/meshes/head_upper_high.stl scale=1 1 1
- link MP_NECK: geometry collision mesh filename=package://minibot_description/meshes/head_lower_low.stl scale=1 1 1; visual mesh filename=package://minibot_description/meshes/head_lower_high.stl scale=1 1 1
- link MP_PELVIS_L: geometry collision mesh filename=package://minibot_description/meshes/yaw_con_low.stl scale=1 1 1; visual mesh filename=package://minibot_description/meshes/yaw_con_high.stl scale=1 1 1
- link MP_PELVIS_R: geometry collision mesh filename=package://minibot_description/meshes/yaw_con_low.stl scale=1 1 1; visual mesh filename=package://minibot_description/meshes/yaw_con_high.stl scale=1 1 1
- link MP_THIGH1_L: geometry collision mesh filename=package://minibot_description/meshes/hip_roll_low.stl scale=1 1 1; visual mesh filename=package://minibot_description/meshes/hip_roll_high.stl scale=1 1 1
- link MP_THIGH1_R: geometry collision mesh filename=package://minibot_description/meshes/hip_roll_low.stl scale=1 1 1; visual mesh filename=package://minibot_description/meshes/hip_roll_high.stl scale=1 1 1
- link MP_THIGH2_L: geometry collision mesh filename=package://minibot_description/meshes/upper_leg_low.stl scale=1 1 1; visual mesh filename=package://minibot_description/meshes/upper_leg_high.stl scale=1 1 1
- link MP_THIGH2_R: geometry collision mesh filename=package://minibot_description/meshes/upper_leg_low.stl scale=1 1 1; visual mesh filename=package://minibot_description/meshes/upper_leg_high.stl scale=1 1 1
- link MP_TIBIA_L: geometry collision mesh filename=package://minibot_description/meshes/lower_leg_low.stl scale=1 1 1; visual mesh filename=package://minibot_description/meshes/lower_leg_high.stl scale=1 1 1
- link MP_TIBIA_R: geometry collision mesh filename=package://minibot_description/meshes/lower_leg_low.stl scale=1 1 1; visual mesh filename=package://minibot_description/meshes/lower_leg_high.stl scale=1 1 1
Joints:
- joint HeadPan: origin xyz=0 0 0.0235 rpy=0 0 1.5707963 -> xyz=0 0 0.050593 rpy=0 0 1.5707963
- joint LAnklePitch: origin xyz=-0.093 0 0 rpy=3.14159 0 0 -> xyz=-0.150 0 0 rpy=3.14159 0 0
- joint LElbow: origin xyz=-0.06 0 -0.016 rpy=-1.5707963 3.14159 0 -> xyz=-0.14 0 0 rpy=-1.5707963 3.14159 0
- joint LHipRoll: origin xyz=0 0 0.028652 rpy=1.5707963 0 0 -> xyz=0 0 0.038444 rpy=1.5707963 0 0
- joint LHipYaw: origin xyz=-0.005 0.037 -0.09355 rpy=0 3.14159 -1.5707963 -> xyz=-0.022 0.057775 -0.160593 rpy=0 3.14159 -1.5707963
- joint LKnee: origin xyz=-0.093 0 0 rpy=0 0 0 -> xyz=-0.150 0 0 rpy=0 0 0
- joint LShoulderRoll: origin xyz=-0.016 0 0.02165 rpy=1.5707963 1.5707963 0 -> xyz=0 0 0.029194 rpy=1.5707963 1.5707963 0
- joint RAnklePitch: origin xyz=0.093 0 0 rpy=3.14159 0 0 -> xyz=0.150 0 0 rpy=3.14159 0 0
- joint RElbow: origin xyz=-0.06 0 0.016 rpy=-1.5707963 3.14159 0 -> xyz=-0.14 0 0 rpy=-1.5707963 3.14159 0
- joint RHipRoll: origin xyz=0 0 0.028652 rpy=-1.5707963 0 0 -> xyz=0 0 0.038444 rpy=-1.5707963 0 0
- joint RHipYaw: origin xyz=-0.005 -0.037 -0.09355 rpy=0 3.14159 1.5707963 -> xyz=-0.022 -0.057775 -0.160593 rpy=0 3.14159 1.5707963
- joint RKnee: origin xyz=0.093 0 0 rpy=0 0 0 -> xyz=0.150 0 0 rpy=0 0 0
- joint base_link_to_body: origin xyz=0 0 0 rpy=0 0 0 -> xyz=0 0 1 rpy=0 0 0

Commit message: fixed collision model and camera position

File: urdf/minibot.urdf (robot description, URDF)
Before this commit: robot Minibot, 25 links, 24 joints
Links:
- added link MP_IMU
- link MP_ARM_HIGH_L: geometry collision mesh filename=package://minibot_description/meshes/upper_arm_high.stl scale=1 1 1; visual mesh filename=package://minibot_description/meshes/upper_arm_high.stl scale=1 1 1
- link MP_THIGH2_L: geometry collision mesh filename=package://minibot_description/meshes/upper_leg_high.stl scale=1 1 1; visual mesh filename=package://minibot_description/meshes/upper_leg_high.stl scale=1 1 1
- link MP_THIGH2_R: geometry collision mesh filename=package://minibot_description/meshes/upper_leg_high.stl scale=1 1 1; visual mesh filename=package://minibot_description/meshes/upper_leg_high.stl scale=1 1 1
Joints:
- added joint j_imu: type fixed, parent MP_BODY, child MP_IMU, origin xyz=-0.03 0 -0.05 rpy=0 0 0, axis 0 0 1
- joint base_link_to_body: origin xyz=0 0 1 rpy=0 0 0 -> xyz=0 0 0.6 rpy=0 0 0
- joint j_camboard: limit lower=-2.6179939 upper=2.6179939 effort=2.8 velocity=5.6548668 -> (none); origin xyz=0 0 0.0235 rpy=3.14159 1.5707963 0 -> xyz=0 -0.055 0  rpy=3.14159 3.14159 0

Commit message: newer version from other git

File: urdf/minibot.urdf (robot description, URDF)
Before this commit: robot Minibot, 26 links, 25 joints
Links:
- removed link MP_ANKLE1_L
- removed link MP_ANKLE1_R
- removed link MP_ANKLE2_L
- removed link MP_ANKLE2_R
- removed link MP_ARM_HIGH_L
- removed link MP_ARM_HIGH_R
- removed link MP_ARM_LOW_L
- removed link MP_ARM_LOW_R
- removed link MP_BACK_L
- removed link MP_BACK_R
- removed link MP_BODY
- removed link MP_HEAD
- removed link MP_IMU
- removed link MP_NECK
- removed link MP_PELVIS_L
- removed link MP_PELVIS_R
- removed link MP_PMDCAMBOARD
- removed link MP_SHOULDER_L
- removed link MP_SHOULDER_R
- removed link MP_THIGH1_L
- removed link MP_THIGH1_R
- removed link MP_THIGH2_L
- removed link MP_THIGH2_R
- removed link MP_TIBIA_L
- removed link MP_TIBIA_R
- added link L_ANKLE_PITCH_L, mass 0.325; collision mesh filename=package://minibot_description/meshes/ankle_roll_low.dae scale=1 1 1; visual mesh filename=package://minibot_description/meshes/ankle_roll_low.dae scale=1 1 1
- added link L_ANKLE_PITCH_R, mass 0.325; collision mesh filename=package://minibot_description/meshes/ankle_roll_low.dae scale=1 1 1; visual mesh filename=package://minibot_description/meshes/ankle_roll_low.dae scale=1 1 1
- added link L_ANKLE_ROLL_L, mass 0.086; collision mesh filename=package://minibot_description/meshes/foot_low.stl scale=1 1 1; visual mesh filename=package://minibot_description/meshes/foot_high.stl scale=1 1 1
- added link L_ANKLE_ROLL_R, mass 0.086; collision mesh filename=package://minibot_description/meshes/foot_low.stl scale=1 1 1; visual mesh filename=package://minibot_description/meshes/foot_high.stl scale=1 1 1
- added link L_CAMERA
- added link L_ELBOW_L, mass 0.097; collision mesh filename=package://minibot_description/meshes/lower_arm_low.stl scale=1 1 1; visual mesh filename=package://minibot_description/meshes/lower_arm_high.stl scale=1 1 1
- added link L_ELBOW_R, mass 0.097; collision mesh filename=package://minibot_description/meshes/lower_arm_low.stl scale=1 1 1; visual mesh filename=package://minibot_description/meshes/lower_arm_high.stl scale=1 1 1
- added link L_FOOT_BOTTOM_L
- added link L_FOOT_BOTTOM_R
- added link L_FOOT_FRONT_L
- added link L_FOOT_FRONT_R
- added link L_HEAD_PAN, mass 0.012; collision mesh filename=package://minibot_description/meshes/head_lower_low.stl scale=1 1 1; visual mesh filename=package://minibot_description/meshes/head_lower_high.stl scale=1 1 1
- added link L_HEAD_TILT, mass 0.139; collision mesh filename=package://minibot_description/meshes/head_upper_low.stl scale=1 1 1; visual mesh filename=package://minibot_description/meshes/head_upper_high.stl scale=1 1 1
- added link L_HIP_PITCH_L, mass 0.215; collision mesh filename=package://minibot_description/meshes/upper_leg_high.stl scale=1 1 1; visual mesh filename=package://minibot_description/meshes/upper_leg_high.stl scale=1 1 1
- added link L_HIP_PITCH_R, mass 0.215; collision mesh filename=package://minibot_description/meshes/upper_leg_high.stl scale=1 1 1; visual mesh filename=package://minibot_description/meshes/upper_leg_high.stl scale=1 1 1
- added link L_HIP_ROLL_L, mass 0.325; collision mesh filename=package://minibot_description/meshes/hip_roll_low.dae scale=1 1 1; visual mesh filename=package://minibot_description/meshes/hip_roll_low.dae scale=1 1 1
- added link L_HIP_ROLL_R, mass 0.325; collision mesh filename=package://minibot_description/meshes/hip_roll_low.dae scale=1 1 1; visual mesh filename=package://minibot_description/meshes/hip_roll_low.dae scale=1 1 1
- added link L_HIP_YAW_L, mass 0.022; collision mesh filename=package://minibot_description/meshes/yaw_con_low.stl scale=1 1 1; visual mesh filename=package://minibot_description/meshes/yaw_con_high.stl scale=1 1 1
- added link L_HIP_YAW_R, mass 0.022; collision mesh filename=package://minibot_description/meshes/yaw_con_low.stl scale=1 1 1; visual mesh filename=package://minibot_description/meshes/yaw_con_high.stl scale=1 1 1
- added link L_Hand_L
- added link L_Hand_R
- added link L_IMU
- added link L_KNEE_L, mass 0.055; collision mesh filename=package://minibot_description/meshes/lower_leg_low.stl scale=1 1 1; visual mesh filename=package://minibot_description/meshes/lower_leg_high.stl scale=1 1 1
- added link L_KNEE_R, mass 0.055; collision mesh filename=package://minibot_description/meshes/lower_leg_low.stl scale=1 1 1; visual mesh filename=package://minibot_description/meshes/lower_leg_high.stl scale=1 1 1
- added link L_SHOULDER_PITCH_L, mass 0.018; collision mesh filename=package://minibot_description/meshes/shoulder_con_low.stl scale=1 1 1; visual mesh filename=package://minibot_description/meshes/shoulder_con_high.stl scale=1 1 1
- added link L_SHOULDER_PITCH_R, mass 0.018; collision mesh filename=package://minibot_description/meshes/shoulder_con_low.stl scale=1 1 1; visual mesh filename=package://minibot_description/meshes/shoulder_con_high.stl scale=1 1 1
- added link L_SHOULDER_ROLL_L, mass 0.190; collision mesh filename=package://minibot_description/meshes/upper_arm_high.dae scale=1 1 1; visual mesh filename=package://minibot_description/meshes/upper_arm_high.dae scale=1 1 1
- added link L_SHOULDER_ROLL_R, mass 0.190; collision mesh filename=package://minibot_description/meshes/upper_arm_high.dae scale=1 1 1; visual mesh filename=package://minibot_description/meshes/upper_arm_high.dae scale=1 1 1
- added link L_TORSO, mass 1.423; collision mesh filename=package://minibot_description/meshes/torso_low.dae scale=1 1 1; visual mesh filename=package://minibot_description/meshes/torso_low.dae scale=1 1 1
Joints:
- removed joint j_back_l
- removed joint j_back_r
- added joint j_LFootBottom: type fixed, parent L_ANKLE_ROLL_L, child L_FOOT_BOTTOM_L, origin xyz=-0.040444 0 0 rpy=3.14159 -1.5707963 0
- added joint j_LFootFront: type fixed, parent L_FOOT_BOTTOM_L, child L_FOOT_FRONT_L, origin xyz=0.0849 0 0 
- added joint j_LHand: type fixed, parent L_ELBOW_L, child L_Hand_L, origin xyz=-0.1573 0 0 rpy=0 0 3.14159
- added joint j_RFootBottom: type fixed, parent L_ANKLE_ROLL_R, child L_FOOT_BOTTOM_R, origin xyz=0.040444 0 0 rpy=0 -1.5707963 0
- added joint j_RFootFront: type fixed, parent L_FOOT_BOTTOM_R, child L_FOOT_FRONT_R, origin xyz=0.0849 0 0 
- added joint j_RHand: type fixed, parent L_ELBOW_R, child L_Hand_R, origin xyz=0.1573 0 0
- joint HeadPan: child MP_NECK -> L_HEAD_PAN; limit lower=-2.6179939 upper=2.6179939 effort=2.8 velocity=5.6548668 -> lower=-2.1816615649875 upper=2.1816615649875 effort=2.5 velocity=5.6548668; parent MP_BODY -> L_TORSO
- joint HeadTilt: child MP_HEAD -> L_HEAD_TILT; limit lower=-2.6179939 upper=2.6179939 effort=2.8 velocity=5.6548668 -> lower=-1.5707963267910001 upper=0 effort=2.5 velocity=5.6548668; parent MP_NECK -> L_HEAD_PAN
- joint LAnklePitch: axis 0 0 1 -> 0 0 -1; child MP_ANKLE1_L -> L_ANKLE_PITCH_L; limit lower=-2.6179939 upper=2.6179939 effort=10 velocity=5.6548668 -> lower=-1.6406094968706 upper=1.2391837689129 effort=8.4 velocity=4.712388975; parent MP_TIBIA_L -> L_KNEE_L
- joint LAnkleRoll: child MP_ANKLE2_L -> L_ANKLE_ROLL_L; limit lower=-2.6179939 upper=2.6179939 effort=10 velocity=5.6548668 -> lower=-1.4660765716716 upper=1.4660765716716 effort=6.0 velocity=6.597344565; parent MP_ANKLE1_L -> L_ANKLE_PITCH_L
- joint LElbow: child MP_ARM_LOW_L -> L_ELBOW_L; limit lower=-2.6179939 upper=2.6179939 effort=2.8 velocity=5.6548668 -> lower=-1.1344640137935 upper=1.5707963267910001 effort=2.5 velocity=5.6548668; origin xyz=-0.14 0 0 rpy=-1.5707963 3.14159 0 -> xyz=-0.14 0 0 rpy=1.5707963 1.5707963 0; parent MP_ARM_HIGH_L -> L_SHOULDER_ROLL_L
- joint LHipPitch: child MP_THIGH2_L -> L_HIP_PITCH_L; limit lower=-2.6179939 upper=2.6179939 effort=10 velocity=5.6548668 -> lower=-0.48869219055720003 upper=1.919862177189 effort=8.4 velocity=4.712388975; origin xyz=0 0 0 rpy=1.5707963 0 -1.5707963 -> xyz=0 0 0 rpy=1.5707963 0 1.5707963; parent MP_THIGH1_L -> L_HIP_ROLL_L
- joint LHipRoll: axis 0 0 1 -> 0 0 -1; child MP_THIGH1_L -> L_HIP_ROLL_L; limit lower=-2.6179939 upper=2.6179939 effort=10 velocity=5.6548668 -> lower=-1.0122909661542001 upper=0.7853981633955001 effort=6.0 velocity=6.597344565; origin xyz=0 0 0.038444 rpy=1.5707963 0 0 -> xyz=0 0 0.038444 rpy=-1.5707963 0 1.5707963; parent MP_PELVIS_L -> L_HIP_YAW_L
- joint LHipYaw: child MP_PELVIS_L -> L_HIP_YAW_L; limit lower=-2.6179939 upper=2.6179939 effort=10 velocity=5.6548668 -> lower=-0.9250245035547 upper=0.9250245035547 effort=2.5 velocity=5.6548668; origin xyz=-0.022 0.057775 -0.160593 rpy=0 3.14159 -1.5707963 -> xyz=-0.022 0.057775 -0.160593 rpy=0 3.14159 3.14159; parent MP_BODY -> L_TORSO
- joint LKnee: child MP_TIBIA_L -> L_KNEE_L; limit lower=-2.6179939 upper=2.6179939 effort=10 velocity=5.6548668 -> lower=-2.268928027587 upper=0 effort=8.4 velocity=4.712388975; parent MP_THIGH2_L -> L_HIP_PITCH_L
- joint LShoulderPitch: child MP_SHOULDER_L -> L_SHOULDER_PITCH_L; limit lower=-2.6179939 upper=2.6179939 effort=2.8 velocity=5.6548668 -> lower=-3.1415926535820002 upper=3.1415926535820002 effort=6.0 velocity=6.597344565; origin xyz=0 0 0 rpy=0 0 -1.5707963 -> xyz=0 0.08134 0 rpy=0 -1.5707963 -1.5707963; parent MP_BACK_L -> L_TORSO
- joint LShoulderRoll: axis 0 0 1 -> 0 0 -1; child MP_ARM_HIGH_L -> L_SHOULDER_ROLL_L; limit lower=-2.6179939 upper=2.6179939 effort=2.8 velocity=5.648668 -> lower=-2.3561944901865 upper=0.7853981633955001 effort=2.5 velocity=5.648668; origin xyz=0 0 0.029194 rpy=1.5707963 1.5707963 0 -> xyz=0 0 0.029194 rpy=-1.5707963 0.7853981633955001 0; parent MP_SHOULDER_L -> L_SHOULDER_PITCH_L
- joint RAnklePitch: axis 0 0 1 -> 0 0 -1; child MP_ANKLE1_R -> L_ANKLE_PITCH_R; limit lower=-2.6179939 upper=2.6179939 effort=10 velocity=5.6548668 -> lower=-1.2391837689129 upper=1.6406094968706 effort=8.4 velocity=4.712388975; parent MP_TIBIA_R -> L_KNEE_R
- joint RAnkleRoll: child MP_ANKLE2_R -> L_ANKLE_ROLL_R; limit lower=-2.6179939 upper=2.6179939 effort=10 velocity=5.6548668 -> lower=-1.4660765716716 upper=1.4660765716716 effort=6.0 velocity=6.597344565; parent MP_ANKLE1_R -> L_ANKLE_PITCH_R
- joint RElbow: child MP_ARM_LOW_R -> L_ELBOW_R; limit lower=-1.635 upper=2.6179939 effort=2.8 velocity=5.6548668 -> lower=-1.635 upper=1.5707963267910001 effort=2.5 velocity=5.6548668; origin xyz=-0.14 0 0 rpy=-1.5707963 3.14159 0 -> xyz=-0.14 0 0 rpy=-1.5707963 -1.5707963 0; parent MP_ARM_HIGH_R -> L_SHOULDER_ROLL_R
- joint RHipPitch: child MP_THIGH2_R -> L_HIP_PITCH_R; limit lower=-2.6179939 upper=2.6179939 effort=10 velocity=5.6548668 -> lower=-1.919862177189 upper=0.48869219055720003 effort=8.4 velocity=4.712388975; parent MP_THIGH1_R -> L_HIP_ROLL_R
- joint RHipRoll: child MP_THIGH1_R -> L_HIP_ROLL_R; limit lower=-2.6179939 upper=2.6179939 effort=10 velocity=5.6548668 -> lower=-1.0122909661542001 upper=0.7853981633955001 effort=6.0 velocity=6.597344565; origin xyz=0 0 0.038444 rpy=-1.5707963 0 0 -> xyz=0 0 0.038444 rpy=-1.5707963 0 1.5707963; parent MP_PELVIS_R -> L_HIP_YAW_R
- joint RHipYaw: child MP_PELVIS_R -> L_HIP_YAW_R; limit lower=-2.6179939 upper=2.6179939 effort=10 velocity=5.6548668 -> lower=-0.9250245035547 upper=0.9250245035547 effort=2.5 velocity=5.6548668; origin xyz=-0.022 -0.057775 -0.160593 rpy=0 3.14159 1.5707963 -> xyz=-0.022 -0.057775 -0.160593 rpy=0 3.14159 3.14159; parent MP_BODY -> L_TORSO
- joint RKnee: child MP_TIBIA_R -> L_KNEE_R; limit lower=-2.6179939 upper=2.6179939 effort=10 velocity=5.6548668 -> lower=-2.268928027587 upper=0 effort=8.4 velocity=4.712388975; parent MP_THIGH2_R -> L_HIP_PITCH_R
- joint RShoulderPitch: child MP_SHOULDER_R -> L_SHOULDER_PITCH_R; limit lower=-2.6179939 upper=2.6179939 effort=2.8 velocity=5.6548668 -> lower=-3.1415926535820002 upper=3.1415926535820002 effort=6.0 velocity=6.597344565; origin xyz=0 0 0 rpy=0 0 -1.5707963 -> xyz=0 -0.08134 0 rpy=0 1.5707963 -1.5707963; parent MP_BACK_R -> L_TORSO
- joint RShoulderRoll: axis 0 0 1 -> 0 0 -1; child MP_ARM_HIGH_R -> L_SHOULDER_ROLL_R; limit lower=-2.6179939 upper=2.6179939 effort=2.8 velocity=5.648668 -> lower=-0.7853981633955001 upper=2.3561944901865 effort=2.5 velocity=5.648668; origin xyz=0 0 0.029194 rpy=-1.5707963 1.5707963 0 -> xyz=0 0 0.029194 rpy=-1.5707963 2.356194463 0; parent MP_SHOULDER_R -> L_SHOULDER_PITCH_R
- joint base_link_to_body: child MP_BODY -> L_TORSO; origin xyz=0 0 0.6 rpy=0 0 0 -> xyz=0 0 0.58 rpy=0 0 0
- joint j_camboard: child MP_PMDCAMBOARD -> L_CAMERA; origin xyz=0 -0.055 0  rpy=3.14159 3.14159 0 -> xyz=0 -0.055 0  rpy=-1.5707963 0 3.14159; parent MP_HEAD -> L_HEAD_TILT
- joint j_imu: child MP_IMU -> L_IMU; parent MP_BODY -> L_TORSO
