Commit message: added readme und updated some stuff

File: urdf/minibot.urdf.xacro (robot description, xacro)
@@ -306,5 +306,5 @@
       <mass value="0.055"/>
       <!--<inertia ixx="0.000094062"  ixy="0.0"  ixz="0.0" iyy="0.000043139" iyz="-0.000002344" izz="0.000125827" />-->
-      <inertia ixx="${insu+infa*0.000094062}"  ixy="0"  ixz="0" iyy="${insu+infa*0.000043139}" iyz="0" izz="${insu+infa*0.000125827}" />
+      <inertia ixx="${insu*0.1+infa*0.000094062}"  ixy="0"  ixz="0" iyy="${insu*0.1+infa*0.000043139}" iyz="0" izz="${insu*0.1+infa*0.000125827}" />
       <!--<inertia ixx="0.001"  ixy="0.001"  ixz="0.001" iyy="0.001" iyz="0.001" izz="0.001" />-->
     </inertial>
@@ -454,5 +454,5 @@
       <mass value="0.055"/>
       <!--<inertia ixx="0.000094062"  ixy="0.0"  ixz="0.0" iyy="0.000043139" iyz="-0.000002344" izz="0.000125827" />-->
-      <inertia ixx="${insu+infa*0.000094062}"  ixy="0"  ixz="0" iyy="${insu+infa*0.000043139}" iyz="0" izz="${insu+infa*0.000125827}" />
+      <inertia ixx="${insu*0.1+infa*0.000094062}"  ixy="0"  ixz="0" iyy="${insu*0.1+infa*0.000043139}" iyz="0" izz="${insu*0.1+infa*0.000125827}" />
       <!--<inertia ixx="0.001"  ixy="0.001"  ixz="0.001" iyy="0.001" iyz="0.001" izz="0.001" />-->
     </inertial>
