Commit message: Beim Minibot Die Position der Roll und Pitchmotoren in den Beinen genauer gemacht

File: minibot_description/urdf/minibot.urdf (robot description, URDF)
Before this commit: robot Minibot, 30 links, 29 joints
Joints:
- joint LAnkleRoll: origin xyz=0 0 0 rpy=-1.5707963 0 0 -> xyz=0 -0.025 0 rpy=-1.5707963 0 0
- joint LHipPitch: origin xyz=0 0 0 rpy=1.5707963 0 1.5707963 -> xyz=0 0 -0.025 rpy=1.5707963 0 1.5707963
- joint LHipRoll: origin xyz=0 0 0.038444 rpy=-1.5707963 0 1.5707963 -> xyz=-0.025 0 0.038444 rpy=-1.5707963 0 1.5707963
- joint RAnkleRoll: origin xyz=0 0 0 rpy=-1.5707963 0 0 -> xyz=0 -0.025 0 rpy=-1.5707963 0 0
- joint RHipPitch: origin xyz=0 0 0 rpy=1.5707963 0 -1.5707963 -> xyz=0 0 -0.025 rpy=1.5707963 0 -1.5707963
- joint RHipRoll: origin xyz=0 0 0.038444 rpy=-1.5707963 0 1.5707963 -> xyz=-0.025 0 0.038444 rpy=-1.5707963 0 1.5707963

File: minibot_description/urdf/minibot.urdf.xacro (robot description, xacro)
@@ -260,5 +260,5 @@
     </inertial>
     <visual>
-      <origin xyz="0 0 0" rpy="0 3.14 0" />
+      <origin xyz="0 0 -0.025" rpy="0 3.14 0" />
       <geometry>
         <!--box size="0.001 0.001 0.001"/-->
@@ -270,5 +270,5 @@
     </visual>
     <collision>
-      <origin xyz="0 0 0" rpy="0 3.14 0" />
+      <origin xyz="0 0 -0.025" rpy="0 3.14 0" />
       <geometry>
         <mesh filename="package://minibot_description/meshes/hip_roll_coll.dae"  scale="1 1 1"/>
@@ -359,5 +359,5 @@
     </inertial>
     <visual>
-      <origin xyz="0 0 0" rpy="0 0 -1.5707963268" />
+      <origin xyz="0 0 -0.025" rpy="0 0 -1.5707963268" />
       <geometry>
         <!--box size="0.008 0.066 0.104"/-->
@@ -369,5 +369,5 @@
     </visual>
     <collision>
-      <origin xyz="0 0 0" rpy="0 0 -1.5707963268" />
+      <origin xyz="0 0 -0.025" rpy="0 0 -1.5707963268" />
       <geometry>
         <mesh filename="package://minibot_description/meshes/foot_coll.dae"  scale="1 1 1"/>
@@ -408,5 +408,5 @@
     </inertial>
     <visual>
-      <origin xyz="0 0 0" rpy="0 3.14 0" />
+      <origin xyz="0 0 -0.025" rpy="0 3.14 0" />
       <geometry>
         <!--box size="0.001 0.001 0.001"/-->
@@ -418,5 +418,5 @@
     </visual>
     <collision>
-      <origin xyz="0 0 0" rpy="0 3.14 0" />
+      <origin xyz="0 0 -0.025" rpy="0 3.14 0" />
       <geometry>
         <mesh filename="package://minibot_description/meshes/hip_roll_coll.dae"  scale="1 1 1"/>
@@ -507,5 +507,5 @@
     </inertial>
     <visual>
-      <origin xyz="0 0 0" rpy="0 0 1.5707963268" />
+      <origin xyz="0 0 -0.025" rpy="0 0 1.5707963268" />
       <geometry>
         <!--box size="0.008 0.066 0.104"/-->
@@ -517,5 +517,5 @@
     </visual>
     <collision>
-      <origin xyz="0 0 0" rpy="0 0 1.5707963268" />
+      <origin xyz="0 0 -0.025" rpy="0 0 1.5707963268" />
       <geometry>
         <mesh filename="package://minibot_description/meshes/foot_coll.dae"  scale="1 1 1"/>
@@ -620,5 +620,5 @@
     <parent link="L_HIP_YAW_L"/>
     <child link="L_HIP_ROLL_L"/>
-    <origin xyz="0 0 0.038444" rpy="-1.5707963 0 1.5707963" />
+    <origin xyz="-0.025 0 0.038444" rpy="-1.5707963 0 1.5707963" />
     <axis xyz="0 0 -1" />
     <limit effort="${tofa*6.0}" velocity="6.597344565" lower="-1.0122909661542001" upper="0.7853981633955001" />
@@ -627,5 +627,5 @@
     <parent link="L_HIP_ROLL_L"/>
     <child link="L_HIP_PITCH_L"/>
-    <origin xyz="0 0 0" rpy="1.5707963 0 1.5707963" />
+    <origin xyz="0 0 -0.025" rpy="1.5707963 0 1.5707963" />
     <axis xyz="0 0 1" />
     <limit effort="${tofa*8.4}" velocity="4.712388975" lower="-0.48869219055720003" upper="1.919862177189" />
@@ -648,5 +648,5 @@
     <parent link="L_ANKLE_PITCH_L"/>
     <child link="L_ANKLE_ROLL_L"/>
-    <origin xyz="0 0 0" rpy="-1.5707963 0 0" />
+    <origin xyz="0 -0.025 0" rpy="-1.5707963 0 0" />
     <axis xyz="0 0 1" />
     <limit effort="${tofa*6.0}" velocity="6.597344565" lower="-1.4660765716716" upper="1.4660765716716" />
@@ -672,5 +672,5 @@
     <parent link="L_HIP_YAW_R"/>
     <child link="L_HIP_ROLL_R"/>
-    <origin xyz="0 0 0.038444" rpy="-1.5707963 0 1.5707963" />
+    <origin xyz="-0.025 0 0.038444" rpy="-1.5707963 0 1.5707963" />
     <axis xyz="0 0 1" />
     <limit effort="${tofa*6.0}" velocity="6.597344565" lower="-1.0122909661542001" upper="0.7853981633955001" />
@@ -679,5 +679,5 @@
     <parent link="L_HIP_ROLL_R"/>
     <child link="L_HIP_PITCH_R"/>
-    <origin xyz="0 0 0" rpy="1.5707963 0 -1.5707963" />
+    <origin xyz="0 0 -0.025" rpy="1.5707963 0 -1.5707963" />
     <axis xyz="0 0 1" />
     <limit effort="${tofa*8.4}" velocity="4.712388975" lower="-1.919862177189" upper="0.48869219055720003" />
@@ -700,5 +700,5 @@
     <parent link="L_ANKLE_PITCH_R"/>
     <child link="L_ANKLE_ROLL_R"/>
-    <origin xyz="0 0 0" rpy="-1.5707963 0 0" />
+    <origin xyz="0 -0.025 0" rpy="-1.5707963 0 0" />
     <axis xyz="0 0 1" />
     <limit effort="${tofa*6.0}" velocity="6.597344565" lower="-1.4660765716716" upper="1.4660765716716" />

Commit message: Minibot Position of Footplate fixed

File: minibot_description/urdf/minibot.urdf (robot description, URDF)
Before this commit: robot Minibot, 30 links, 29 joints
Joints:
- joint LAnkleRoll: origin xyz=0 -0.025 0 rpy=-1.5707963 0 0 -> xyz=0 0.0275 0 rpy=-1.5707963 0 0
- joint RAnkleRoll: origin xyz=0 -0.025 0 rpy=-1.5707963 0 0 -> xyz=0 0.0275 0 rpy=-1.5707963 0 0
- joint RKnee: limit lower=-2.268928027587 upper=0 effort=33.6 velocity=4.712388975 -> lower=0 upper=2.268928027587 effort=33.6 velocity=4.712388975

File: minibot_description/urdf/minibot.urdf.xacro (robot description, xacro)
@@ -648,5 +648,5 @@
     <parent link="L_ANKLE_PITCH_L"/>
     <child link="L_ANKLE_ROLL_L"/>
-    <origin xyz="0 -0.025 0" rpy="-1.5707963 0 0" />
+    <origin xyz="0 0.0275 0" rpy="-1.5707963 0 0" />
     <axis xyz="0 0 1" />
     <limit effort="${tofa*6.0}" velocity="6.597344565" lower="-1.4660765716716" upper="1.4660765716716" />
@@ -688,5 +688,5 @@
     <origin xyz="0.150 0 0" rpy="0 0 0" />
     <axis xyz="0 0 1" />
-    <limit effort="${tofa*8.4}" velocity="4.712388975" lower="-2.268928027587" upper="0" />
+    <limit effort="${tofa*8.4}" velocity="4.712388975" lower="0" upper="2.268928027587" />
   <dynamics damping="${d}" friction="0.0"/> </joint>
   <joint name="RAnklePitch" type="revolute">
@@ -700,5 +700,5 @@
     <parent link="L_ANKLE_PITCH_R"/>
     <child link="L_ANKLE_ROLL_R"/>
-    <origin xyz="0 -0.025 0" rpy="-1.5707963 0 0" />
+    <origin xyz="0 0.0275 0" rpy="-1.5707963 0 0" />
     <axis xyz="0 0 1" />
     <limit effort="${tofa*6.0}" velocity="6.597344565" lower="-1.4660765716716" upper="1.4660765716716" />

Commit message: fixed minibot urdf and added new launch

File: minibot_description/urdf/minibot.urdf (robot description, URDF)
Before this commit: robot Minibot, 30 links, 29 joints
Joints:
- joint LAnklePitch: axis 0 0 -1 -> 0 0 1
- joint LHipPitch: axis 0 0 1 -> 0 0 -1
- joint LKnee: axis 0 0 1 -> 0 0 -1
- joint RHipRoll: axis 0 0 1 -> 0 0 -1
- joint base_link_to_body: origin xyz=0 0 0.545 rpy=0 0 0 -> xyz=0 0 0.545 rpy=0 0.26 0

File: minibot_description/urdf/minibot.urdf.xacro (robot description, xacro)
@@ -10,5 +10,5 @@
     <parent link="base_link"/>
     <child link="L_TORSO"/>
-    <origin xyz="0 0 0.545" rpy="0 0 0" />
+    <origin xyz="0 0 0.545" rpy="0 0.26 0" />
   </joint>
   <link name="L_TORSO">
@@ -628,5 +628,5 @@
     <child link="L_HIP_PITCH_L"/>
     <origin xyz="0 0 -0.025" rpy="1.5707963 0 1.5707963" />
-    <axis xyz="0 0 1" />
+    <axis xyz="0 0 -1" />
     <limit effort="${tofa*8.4}" velocity="4.712388975" lower="-0.48869219055720003" upper="1.919862177189" />
   <dynamics damping="${d}" friction="0.0"/> </joint>
@@ -635,5 +635,5 @@
     <child link="L_KNEE_L"/>
     <origin xyz="-0.150 0 0" rpy="0 0 0" />
-    <axis xyz="0 0 1" />
+    <axis xyz="0 0 -1" />
     <limit effort="${tofa*8.4}" velocity="4.712388975" lower="-2.268928027587" upper="0" />
   <dynamics damping="${d}" friction="0.0"/> </joint>
@@ -642,5 +642,5 @@
     <child link="L_ANKLE_PITCH_L"/>
     <origin xyz="-0.150 0 0" rpy="3.14159 0 0" />
-    <axis xyz="0 0 -1" />
+    <axis xyz="0 0 1" />
     <limit effort="${tofa*8.4}" velocity="4.712388975" lower="-1.6406094968706" upper="1.2391837689129" />
   <dynamics damping="${d}" friction="0.0"/> </joint>
@@ -673,5 +673,5 @@
     <child link="L_HIP_ROLL_R"/>
     <origin xyz="-0.025 0 0.038444" rpy="-1.5707963 0 1.5707963" />
-    <axis xyz="0 0 1" />
+    <axis xyz="0 0 -1" />
     <limit effort="${tofa*6.0}" velocity="6.597344565" lower="-1.0122909661542001" upper="0.7853981633955001" />
   <dynamics damping="${d}" friction="0.0"/> </joint>

Commit message: reverted wrong change in model

File: minibot_description/urdf/minibot.urdf (robot description, URDF)
Before this commit: robot Minibot, 30 links, 29 joints
Joints:
- joint LAnklePitch: axis 0 0 1 -> 0 0 -1
- joint LHipPitch: axis 0 0 -1 -> 0 0 1
- joint LKnee: axis 0 0 -1 -> 0 0 1
- joint RHipRoll: axis 0 0 -1 -> 0 0 1
- joint base_link_to_body: origin xyz=0 0 0.545 rpy=0 0.26 0 -> xyz=0 0 0.545 rpy=0 0 0

File: minibot_description/urdf/minibot.urdf.xacro (robot description, xacro)
@@ -10,5 +10,5 @@
     <parent link="base_link"/>
     <child link="L_TORSO"/>
-    <origin xyz="0 0 0.545" rpy="0 0.26 0" />
+    <origin xyz="0 0 0.545" rpy="0 0 0" />
   </joint>
   <link name="L_TORSO">
@@ -628,5 +628,5 @@
     <child link="L_HIP_PITCH_L"/>
     <origin xyz="0 0 -0.025" rpy="1.5707963 0 1.5707963" />
-    <axis xyz="0 0 -1" />
+    <axis xyz="0 0 1" />
     <limit effort="${tofa*8.4}" velocity="4.712388975" lower="-0.48869219055720003" upper="1.919862177189" />
   <dynamics damping="${d}" friction="0.0"/> </joint>
@@ -635,5 +635,5 @@
     <child link="L_KNEE_L"/>
     <origin xyz="-0.150 0 0" rpy="0 0 0" />
-    <axis xyz="0 0 -1" />
+    <axis xyz="0 0 1" />
     <limit effort="${tofa*8.4}" velocity="4.712388975" lower="-2.268928027587" upper="0" />
   <dynamics damping="${d}" friction="0.0"/> </joint>
@@ -642,5 +642,5 @@
     <child link="L_ANKLE_PITCH_L"/>
     <origin xyz="-0.150 0 0" rpy="3.14159 0 0" />
-    <axis xyz="0 0 1" />
+    <axis xyz="0 0 -1" />
     <limit effort="${tofa*8.4}" velocity="4.712388975" lower="-1.6406094968706" upper="1.2391837689129" />
   <dynamics damping="${d}" friction="0.0"/> </joint>
@@ -673,5 +673,5 @@
     <child link="L_HIP_ROLL_R"/>
     <origin xyz="-0.025 0 0.038444" rpy="-1.5707963 0 1.5707963" />
-    <axis xyz="0 0 -1" />
+    <axis xyz="0 0 1" />
     <limit effort="${tofa*6.0}" velocity="6.597344565" lower="-1.0122909661542001" upper="0.7853981633955001" />
   <dynamics damping="${d}" friction="0.0"/> </joint>

Commit message: fixed urdf

File: minibot_description/urdf/minibot.urdf (robot description, URDF)
Before this commit: robot Minibot, 30 links, 29 joints
Joints:
- joint LAnklePitch: axis 0 0 -1 -> 0 0 1
- joint RAnklePitch: axis 0 0 -1 -> 0 0 1
- joint base_link_to_body: origin xyz=0 0 0.545 rpy=0 0 0 -> xyz=0 0 0.545 rpy=0 0.2 0

File: minibot_description/urdf/minibot.urdf.xacro (robot description, xacro)
@@ -10,5 +10,5 @@
     <parent link="base_link"/>
     <child link="L_TORSO"/>
-    <origin xyz="0 0 0.545" rpy="0 0 0" />
+    <origin xyz="0 0 0.545" rpy="0 0.2 0" />
   </joint>
   <link name="L_TORSO">
@@ -642,5 +642,5 @@
     <child link="L_ANKLE_PITCH_L"/>
     <origin xyz="-0.150 0 0" rpy="3.14159 0 0" />
-    <axis xyz="0 0 -1" />
+    <axis xyz="0 0 1" />
     <limit effort="${tofa*8.4}" velocity="4.712388975" lower="-1.6406094968706" upper="1.2391837689129" />
   <dynamics damping="${d}" friction="0.0"/> </joint>
@@ -694,5 +694,5 @@
     <child link="L_ANKLE_PITCH_R"/>
     <origin xyz="0.150 0 0" rpy="3.14159 0 0" />
-    <axis xyz="0 0 -1" />
+    <axis xyz="0 0 1" />
     <limit effort="${tofa*8.4}" velocity="4.712388975" lower="-1.2391837689129" upper="1.6406094968706" />
   <dynamics damping="${d}" friction="0.0"/> </joint>

Commit message: worked on urdf

File: minibot_description/urdf/minibot.urdf (robot description, URDF)
Before this commit: robot Minibot, 30 links, 29 joints
Links:
- link L_ANKLE_PITCH_L: geometry visual mesh filename=package://minibot_description/meshes/ankle_roll_low.dae scale=1 1 1
- link L_ANKLE_PITCH_R: geometry visual mesh filename=package://minibot_description/meshes/ankle_roll_low.dae scale=1 1 1
- link L_ELBOW_L: geometry visual mesh filename=package://minibot_description/meshes/lower_arm_high.stl scale=1 1 1
- link L_ELBOW_R: geometry visual mesh filename=package://minibot_description/meshes/lower_arm_high.stl scale=1 1 1
- link L_HEAD_PAN: geometry visual mesh filename=package://minibot_description/meshes/head_lower_high.stl scale=1 1 1
- link L_HEAD_TILT: geometry visual mesh filename=package://minibot_description/meshes/head_upper_high.stl scale=1 1 1
- link L_HIP_PITCH_L: geometry visual mesh filename=package://minibot_description/meshes/upper_leg_high.stl scale=1 1 1
- link L_HIP_PITCH_R: geometry visual mesh filename=package://minibot_description/meshes/upper_leg_high.stl scale=1 1 1
- link L_HIP_ROLL_L: geometry visual mesh filename=package://minibot_description/meshes/hip_roll_low.dae scale=1 1 1
- link L_HIP_ROLL_R: geometry visual mesh filename=package://minibot_description/meshes/hip_roll_low.dae scale=1 1 1
- link L_HIP_YAW_L: geometry visual mesh filename=package://minibot_description/meshes/yaw_con_high.stl scale=1 1 1
- link L_HIP_YAW_R: geometry visual mesh filename=package://minibot_description/meshes/yaw_con_high.stl scale=1 1 1
- link L_KNEE_L: geometry visual mesh filename=package://minibot_description/meshes/lower_leg_high.stl scale=1 1 1
- link L_KNEE_R: geometry visual mesh filename=package://minibot_description/meshes/lower_leg_high.stl scale=1 1 1
- link L_SHOULDER_PITCH_L: geometry visual mesh filename=package://minibot_description/meshes/shoulder_con_high.stl scale=1 1 1
- link L_SHOULDER_PITCH_R: geometry visual mesh filename=package://minibot_description/meshes/shoulder_con_high.stl scale=1 1 1
- link L_SHOULDER_ROLL_L: geometry visual mesh filename=package://minibot_description/meshes/upper_arm_high.dae scale=1 1 1
- link L_SHOULDER_ROLL_R: geometry visual mesh filename=package://minibot_description/meshes/upper_arm_high.dae scale=1 1 1
- link L_TORSO: geometry visual mesh filename=package://minibot_description/meshes/torso_low.dae scale=1 1 1

File: minibot_description/urdf/minibot.urdf.xacro (robot description, xacro)
@@ -29,10 +29,10 @@
       </material>
     </visual>
-    <collision>
+    <!-- collision>
       <origin xyz="0 0 0" rpy="1.5707963268 0 1.5707963268"/>
       <geometry>
         <mesh filename="package://minibot_description/meshes/torso_coll.dae"  scale="1 1 1"/>
       </geometry>
-    </collision>
+    </collision> -->
   </link>
   <link name="L_HEAD_PAN">
@@ -53,10 +53,10 @@
       </material>
     </visual>
-    <collision>
+    <!--<collision>
       <origin xyz="0 0 0" rpy="1.5707963268 0 0" />
       <geometry>
         <mesh filename="package://minibot_description/meshes/head_lower_coll.dae"  scale="1 1 1"/>
       </geometry>
-    </collision>
+    </collision>-->
   </link>
   <link name="L_HEAD_TILT">
@@ -76,10 +76,10 @@
       </material>
     </visual>
-    <collision>
+    <!--<collision>
       <origin xyz="0 0 0" rpy="3.14 1.5707963268 0" />
       <geometry>
         <mesh filename="package://minibot_description/meshes/head_upper_coll.dae"  scale="1 1 1"/>
       </geometry>
-    </collision>
+    </collision>-->
   </link>
   <link name="L_SHOULDER_PITCH_L">
@@ -100,10 +100,10 @@
       </material>
     </visual>
-    <collision>
+    <!--<collision>
       <origin xyz="0 0 0" rpy="0 1.5707963268 1.5707963268"/>
       <geometry>
         <mesh filename="package://minibot_description/meshes/shoulder_con_coll.dae"  scale="1 1 1"/>
       </geometry>
-    </collision>
+    </collision>-->
   </link>
   <link name="L_SHOULDER_ROLL_L" >
@@ -124,10 +124,10 @@
       </material>
     </visual>
-    <collision>
+   <!-- <collision>
       <origin xyz="0 0 0" rpy="0 0 -1.5707963268" />
       <geometry>
         <mesh filename="package://minibot_description/meshes/upper_arm_coll.dae"  scale="1 1 1"/>
       </geometry>
-    </collision>
+    </collision>-->
   </link>
   <link name="L_ELBOW_L" >
@@ -147,10 +147,10 @@
       </material>
     </visual>
-    <collision>
+    <!--<collision>
       <origin xyz="0 0 0" rpy="0 1.5707963268 -1.5707963268" />
       <geometry>
         <mesh filename="package://minibot_description/meshes/lower_arm_coll.dae"  scale="1 1 1"/>
       </geometry>
-    </collision>
+    </collision>-->
   </link>
   <link name="L_SHOULDER_PITCH_R" >
@@ -171,10 +171,10 @@
       </material>
     </visual>
-    <collision>
+    <!--<collision>
       <origin xyz="0 0 0" rpy="0 1.5707963268 1.5707963268"/>
       <geometry>
         <mesh filename="package://minibot_description/meshes/shoulder_con_coll.dae"  scale="1 1 1"/>
       </geometry>
-    </collision>
+    </collision>-->
   </link>
   <link name="L_SHOULDER_ROLL_R" >
@@ -196,10 +196,10 @@
       </material>
     </visual>
-    <collision>
+    <!--<collision>
       <origin xyz="0 0 0" rpy="0 0 -1.5707963268" />
       <geometry>
         <mesh filename="package://minibot_description/meshes/upper_arm_coll.dae"  scale="1 1 1"/>
       </geometry>
-    </collision>
+    </collision>-->
   </link>
   <link name="L_ELBOW_R" >
@@ -220,10 +220,10 @@
       </material>
     </visual>
-    <collision>
+    <!--<collision>
       <origin xyz="0 0 0" rpy="0 1.5707963268 1.5707963268" />
       <geometry>
         <mesh filename="package://minibot_description/meshes/lower_arm_coll.dae"  scale="1 1 1"/>
       </geometry>
-    </collision>
+    </collision>-->
   </link>
   <link name="L_HIP_YAW_L" >
@@ -244,10 +244,10 @@
       </material>
     </visual>
-    <collision>
+    <!--<collision>
       <origin xyz="0 0 0" rpy="1.5707963268 0 0" />
       <geometry>
         <mesh filename="package://minibot_description/meshes/yaw_con_coll.dae"  scale="1 1 1"/>
       </geometry>
-    </collision>
+    </collision>-->
   </link>
   <link name="L_HIP_ROLL_L" >
@@ -269,10 +269,10 @@
       </material>
     </visual>
-    <collision>
+    <!--<collision>
       <origin xyz="0 0 -0.025" rpy="0 3.14 0" />
       <geometry>
         <mesh filename="package://minibot_description/meshes/hip_roll_coll.dae"  scale="1 1 1"/>
       </geometry>
-    </collision>
+    </collision>-->
   </link>
   <link name="L_HIP_PITCH_L" >
@@ -294,10 +294,10 @@
       </material>
     </visual>
-    <collision>
+    <!--<collision>
       <origin xyz="0 0 0" rpy="1.5707963268 1.5707963268 0" />
       <geometry>
         <mesh filename="package://minibot_description/meshes/upper_leg_coll.dae"  scale="1 1 1"/>
       </geometry>
-    </collision>
+    </collision>-->
   </link>
   <link name="L_KNEE_L" >
@@ -319,10 +319,10 @@
       </material>
     </visual>
-    <collision>
+    <!--<collision>
       <origin xyz="0 0 0" rpy="1.5707963268 1.5707963268 0" />
       <geometry>
         <mesh filename="package://minibot_description/meshes/lower_leg_coll.dae"  scale="1 1 1"/>
       </geometry>
-    </collision>
+    </collision>-->
   </link>
   <link name="L_ANKLE_PITCH_L" >
@@ -344,10 +344,10 @@
       </material>
     </visual>
-    <collision>
+    <!--<collision>
       <origin xyz="0 0 0" rpy="3.14 -1.5707963268 1.5707963268" />
       <geometry>
         <mesh filename="package://minibot_description/meshes/ankle_roll_coll.dae"  scale="1 1 1"/>
       </geometry>
-    </collision>
+    </collision>-->
   </link>
   <link name="L_ANKLE_ROLL_L" >
@@ -392,10 +392,10 @@
       </material>
     </visual>
-    <collision>
+    <!--<collision>
       <origin xyz="0 0 0" rpy="1.5707963268 0 0" />
       <geometry>
         <mesh filename="package://minibot_description/meshes/yaw_con_coll.dae"  scale="1 1 1"/>
       </geometry>
-    </collision>
+    </collision>-->
   </link>
   <link name="L_HIP_ROLL_R" >
@@ -417,10 +417,10 @@
       </material>
     </visual>
-    <collision>
+    <!--<collision>
       <origin xyz="0 0 -0.025" rpy="0 3.14 0" />
       <geometry>
         <mesh filename="package://minibot_description/meshes/hip_roll_coll.dae"  scale="1 1 1"/>
       </geometry>
-    </collision>
+    </collision>-->
   </link>
   <link name="L_HIP_PITCH_R" >
@@ -442,10 +442,10 @@
       </material>
     </visual>
-    <collision>
+    <!--<collision>
       <origin xyz="0 0 0" rpy="1.5707963268 -1.5707963268 0" />
       <geometry>
         <mesh filename="package://minibot_description/meshes/upper_leg_coll.dae"  scale="1 1 1"/>
       </geometry>
-    </collision>
+    </collision>-->
   </link>
   <link name="L_KNEE_R" >
@@ -467,10 +467,10 @@
       </material>
     </visual>
-    <collision>
+    <!--<collision>
       <origin xyz="0 0 0" rpy="1.5707963268 -1.5707963268 0" />
       <geometry>
         <mesh filename="package://minibot_description/meshes/lower_leg_coll.dae"  scale="1 1 1"/>
       </geometry>
-    </collision>
+    </collision>-->
   </link>
   <link name="L_ANKLE_PITCH_R" >
@@ -492,10 +492,10 @@
       </material>
     </visual>
-    <collision>
+    <!--<collision>
       <origin xyz="0 0 0" rpy="0 1.5707963268 1.5707963268" />
       <geometry>
         <mesh filename="package://minibot_description/meshes/ankle_roll_coll.dae"  scale="1 1 1"/>
       </geometry>
-    </collision>
+    </collision>-->
   </link>
   <link name="L_ANKLE_ROLL_R" >
@@ -1006,5 +1006,5 @@
     </plugin>
   </gazebo>
-  <gazebo reference="L_CAMERA">
+  <!--<gazebo reference="L_CAMERA">
         <sensor name='camera' type='camera'>
           <pose>-0.050000 -0.010000 0.000000 -1.5708 0.000000 -3.141592</pose>
@@ -1038,5 +1038,5 @@
           </plugin>
       </sensor>
-  </gazebo>
+  </gazebo> -->
       <gazebo>
         <plugin filename="libhector_gazebo_ros_imu.so" name="gazebo_ros_imu">
@@ -1068,5 +1068,5 @@
    <!-- fake controller that allows us to move the robot and to get its oposition -->
    <!-- rostopic pub /minibot/cmd_vel geometry_msgs/Twist "{ linear: [ 0.1, 0, 0], angular: [0.2, 0, 0.1] }" -->
-   <gazebo>
+   <!--<gazebo>
     <plugin name="object_controller" filename="libgazebo_ros_planar_move.so">
       <robotNamespace>minibot</robotNamespace>
@@ -1077,4 +1077,4 @@
       <robotBaseFrame>base_link</robotBaseFrame>
     </plugin>
-  </gazebo>
+  </gazebo> -->
 </robot>
