Commit message: added complete collision model to urdf

File: minibot_description/urdf/minibot.urdf (robot description, URDF)
Before this commit: robot Minibot, 30 links, 29 joints
Links:
- link L_ANKLE_PITCH_L: geometry collision mesh filename=package://minibot_description/meshes/ankle_roll_coll.dae scale=1 1 1; visual mesh filename=package://minibot_description/meshes/ankle_roll_low.dae scale=1 1 1
- link L_ANKLE_PITCH_R: geometry collision mesh filename=package://minibot_description/meshes/ankle_roll_coll.dae scale=1 1 1; visual mesh filename=package://minibot_description/meshes/ankle_roll_low.dae scale=1 1 1
- link L_ELBOW_L: geometry collision mesh filename=package://minibot_description/meshes/lower_arm_coll.dae scale=1 1 1; visual mesh filename=package://minibot_description/meshes/lower_arm_high.stl scale=1 1 1
- link L_ELBOW_R: geometry collision mesh filename=package://minibot_description/meshes/lower_arm_coll.dae scale=1 1 1; visual mesh filename=package://minibot_description/meshes/lower_arm_high.stl scale=1 1 1
- link L_HEAD_PAN: geometry collision mesh filename=package://minibot_description/meshes/head_lower_coll.dae scale=1 1 1; visual mesh filename=package://minibot_description/meshes/head_lower_high.stl scale=1 1 1
- link L_HEAD_TILT: geometry collision mesh filename=package://minibot_description/meshes/head_upper_coll.dae scale=1 1 1; visual mesh filename=package://minibot_description/meshes/head_upper_high.stl scale=1 1 1
- link L_HIP_PITCH_L: geometry collision mesh filename=package://minibot_description/meshes/upper_leg_coll.dae scale=1 1 1; visual mesh filename=package://minibot_description/meshes/upper_leg_high.stl scale=1 1 1
- link L_HIP_PITCH_R: geometry collision mesh filename=package://minibot_description/meshes/upper_leg_coll.dae scale=1 1 1; visual mesh filename=package://minibot_description/meshes/upper_leg_high.stl scale=1 1 1
- link L_HIP_ROLL_L: geometry collision mesh filename=package://minibot_description/meshes/hip_roll_coll.dae scale=1 1 1; visual mesh filename=package://minibot_description/meshes/hip_roll_low.dae scale=1 1 1
- link L_HIP_ROLL_R: geometry collision mesh filename=package://minibot_description/meshes/hip_roll_coll.dae scale=1 1 1; visual mesh filename=package://minibot_description/meshes/hip_roll_low.dae scale=1 1 1
- link L_HIP_YAW_L: geometry collision mesh filename=package://minibot_description/meshes/yaw_con_coll.dae scale=1 1 1; visual mesh filename=package://minibot_description/meshes/yaw_con_high.stl scale=1 1 1
- link L_HIP_YAW_R: geometry collision mesh filename=package://minibot_description/meshes/yaw_con_coll.dae scale=1 1 1; visual mesh filename=package://minibot_description/meshes/yaw_con_high.stl scale=1 1 1
- link L_KNEE_L: geometry collision mesh filename=package://minibot_description/meshes/lower_leg_coll.dae scale=1 1 1; visual mesh filename=package://minibot_description/meshes/lower_leg_high.stl scale=1 1 1
- link L_KNEE_R: geometry collision mesh filename=package://minibot_description/meshes/lower_leg_coll.dae scale=1 1 1; visual mesh filename=package://minibot_description/meshes/lower_leg_high.stl scale=1 1 1
- link L_SHOULDER_PITCH_L: geometry collision mesh filename=package://minibot_description/meshes/shoulder_con_coll.dae scale=1 1 1; visual mesh filename=package://minibot_description/meshes/shoulder_con_high.stl scale=1 1 1
- link L_SHOULDER_PITCH_R: geometry collision mesh filename=package://minibot_description/meshes/shoulder_con_coll.dae scale=1 1 1; visual mesh filename=package://minibot_description/meshes/shoulder_con_high.stl scale=1 1 1
- link L_SHOULDER_ROLL_L: geometry collision mesh filename=package://minibot_description/meshes/upper_arm_coll.dae scale=1 1 1; visual mesh filename=package://minibot_description/meshes/upper_arm_high.dae scale=1 1 1
- link L_SHOULDER_ROLL_R: geometry collision mesh filename=package://minibot_description/meshes/upper_arm_coll.dae scale=1 1 1; visual mesh filename=package://minibot_description/meshes/upper_arm_high.dae scale=1 1 1
- link L_TORSO: geometry collision mesh filename=package://minibot_description/meshes/torso_coll.dae scale=1 1 1; visual mesh filename=package://minibot_description/meshes/torso_low.dae scale=1 1 1
Joints:
- joint HeadPan: limit lower=-2.1816615649875 upper=2.1816615649875 effort=10.0 velocity=5.6548668 -> lower=-2.1816615649875 upper=2.1816615649875 effort=2.5 velocity=5.6548668
- joint HeadTilt: limit lower=-1.5707963267910001 upper=0 effort=10.0 velocity=5.6548668 -> lower=-1.5707963267910001 upper=0 effort=2.5 velocity=5.6548668
- joint LAnklePitch: limit lower=-1.6406094968706 upper=1.2391837689129 effort=33.6 velocity=4.712388975 -> lower=-1.6406094968706 upper=1.2391837689129 effort=8.4 velocity=4.712388975
- joint LAnkleRoll: limit lower=-1.4660765716716 upper=1.4660765716716 effort=24.0 velocity=6.597344565 -> lower=-1.4660765716716 upper=1.4660765716716 effort=6.0 velocity=6.597344565
- joint LElbow: limit lower=-1.1344640137935 upper=1.5707963267910001 effort=10.0 velocity=5.6548668 -> lower=-1.1344640137935 upper=1.5707963267910001 effort=2.5 velocity=5.6548668
- joint LHipPitch: limit lower=-0.48869219055720003 upper=1.919862177189 effort=33.6 velocity=4.712388975 -> lower=-0.48869219055720003 upper=1.919862177189 effort=8.4 velocity=4.712388975
- joint LHipRoll: limit lower=-1.0122909661542001 upper=0.7853981633955001 effort=24.0 velocity=6.597344565 -> lower=-1.0122909661542001 upper=0.7853981633955001 effort=6.0 velocity=6.597344565
- joint LHipYaw: limit lower=-0.9250245035547 upper=0.9250245035547 effort=10.0 velocity=5.6548668 -> lower=-0.9250245035547 upper=0.9250245035547 effort=2.5 velocity=5.6548668
- joint LKnee: limit lower=-2.268928027587 upper=0 effort=33.6 velocity=4.712388975 -> lower=-2.268928027587 upper=0 effort=8.4 velocity=4.712388975
- joint LShoulderPitch: limit lower=-3.1415926535820002 upper=3.1415926535820002 effort=24.0 velocity=6.597344565 -> lower=-3.1415926535820002 upper=3.1415926535820002 effort=6.0 velocity=6.597344565
- joint LShoulderRoll: limit lower=-2.3561944901865 upper=0.7853981633955001 effort=10.0 velocity=5.648668 -> lower=-2.3561944901865 upper=0.7853981633955001 effort=2.5 velocity=5.648668
- joint RAnklePitch: limit lower=-1.2391837689129 upper=1.6406094968706 effort=33.6 velocity=4.712388975 -> lower=-1.2391837689129 upper=1.6406094968706 effort=8.4 velocity=4.712388975
- joint RAnkleRoll: limit lower=-1.4660765716716 upper=1.4660765716716 effort=24.0 velocity=6.597344565 -> lower=-1.4660765716716 upper=1.4660765716716 effort=6.0 velocity=6.597344565
- joint RElbow: limit lower=-1.635 upper=1.5707963267910001 effort=10.0 velocity=5.6548668 -> lower=-1.635 upper=1.5707963267910001 effort=2.5 velocity=5.6548668
- joint RHipPitch: limit lower=-1.919862177189 upper=0.48869219055720003 effort=33.6 velocity=4.712388975 -> lower=-1.919862177189 upper=0.48869219055720003 effort=8.4 velocity=4.712388975
- joint RHipRoll: limit lower=-1.0122909661542001 upper=0.7853981633955001 effort=24.0 velocity=6.597344565 -> lower=-1.0122909661542001 upper=0.7853981633955001 effort=6.0 velocity=6.597344565
- joint RHipYaw: limit lower=-0.9250245035547 upper=0.9250245035547 effort=10.0 velocity=5.6548668 -> lower=-0.9250245035547 upper=0.9250245035547 effort=2.5 velocity=5.6548668
- joint RKnee: limit lower=0 upper=2.268928027587 effort=33.6 velocity=4.712388975 -> lower=0 upper=2.268928027587 effort=8.4 velocity=4.712388975
- joint RShoulderPitch: limit lower=-3.1415926535820002 upper=3.1415926535820002 effort=24.0 velocity=6.597344565 -> lower=-3.1415926535820002 upper=3.1415926535820002 effort=6.0 velocity=6.597344565
- joint RShoulderRoll: limit lower=-0.7853981633955001 upper=2.3561944901865 effort=10.0 velocity=5.648668 -> lower=-0.7853981633955001 upper=2.3561944901865 effort=2.5 velocity=5.648668
- joint base_link_to_body: origin xyz=0 0 0.545 rpy=0 0.2 0 -> xyz=0 0 0.545 rpy=0 0 0

File: minibot_description/urdf/minibot.urdf.xacro (robot description, xacro)
@@ -1,7 +1,7 @@
 <?xml version="1.0" ?>
 <robot name="Minibot" xmlns:xacro="http://www.ros.org/wiki/xacro">
-<xacro:property name="tofa" value="4" /> <!--Torque factor-->
-<xacro:property name="infa" value="0" /> <!--inertia factor-->
-<xacro:property name="insu" value="0.005" /> <!--inertia summand-->
+<xacro:property name="tofa" value="1" /> <!--Torque factor-->
+<xacro:property name="infa" value="1" /> <!--inertia factor-->
+<xacro:property name="insu" value="0" /> <!--inertia summand-->
 <xacro:property name="d" value="0" /> <!-- damping -->
 <xacro:property name="f" value="0" /> <!-- friction -->
@@ -10,5 +10,5 @@
     <parent link="base_link"/>
     <child link="L_TORSO"/>
-    <origin xyz="0 0 0.545" rpy="0 0.2 0" />
+    <origin xyz="0 0 0.545" rpy="0 0 0" />
   </joint>
   <link name="L_TORSO">
@@ -29,5 +29,5 @@
       </material>
     </visual>
-    <!-- collision>
+    <collision>
       <origin xyz="0 0 0" rpy="1.5707963268 0 1.5707963268"/>
       <geometry>
@@ -53,10 +53,10 @@
       </material>
     </visual>
-    <!--<collision>
+    <collision>
       <origin xyz="0 0 0" rpy="1.5707963268 0 0" />
       <geometry>
         <mesh filename="package://minibot_description/meshes/head_lower_coll.dae"  scale="1 1 1"/>
       </geometry>
-    </collision>-->
+    </collision>
   </link>
   <link name="L_HEAD_TILT">
@@ -76,10 +76,10 @@
       </material>
     </visual>
-    <!--<collision>
+    <collision>
       <origin xyz="0 0 0" rpy="3.14 1.5707963268 0" />
       <geometry>
         <mesh filename="package://minibot_description/meshes/head_upper_coll.dae"  scale="1 1 1"/>
       </geometry>
-    </collision>-->
+    </collision>
   </link>
   <link name="L_SHOULDER_PITCH_L">
@@ -100,10 +100,10 @@
       </material>
     </visual>
-    <!--<collision>
+    <collision>
       <origin xyz="0 0 0" rpy="0 1.5707963268 1.5707963268"/>
       <geometry>
         <mesh filename="package://minibot_description/meshes/shoulder_con_coll.dae"  scale="1 1 1"/>
       </geometry>
-    </collision>-->
+    </collision>
   </link>
   <link name="L_SHOULDER_ROLL_L" >
@@ -124,10 +124,10 @@
       </material>
     </visual>
-   <!-- <collision>
+   <collision>
       <origin xyz="0 0 0" rpy="0 0 -1.5707963268" />
       <geometry>
         <mesh filename="package://minibot_description/meshes/upper_arm_coll.dae"  scale="1 1 1"/>
       </geometry>
-    </collision>-->
+    </collision>
   </link>
   <link name="L_ELBOW_L" >
@@ -147,10 +147,10 @@
       </material>
     </visual>
-    <!--<collision>
+    <collision>
       <origin xyz="0 0 0" rpy="0 1.5707963268 -1.5707963268" />
       <geometry>
         <mesh filename="package://minibot_description/meshes/lower_arm_coll.dae"  scale="1 1 1"/>
       </geometry>
-    </collision>-->
+    </collision>
   </link>
   <link name="L_SHOULDER_PITCH_R" >
@@ -171,10 +171,10 @@
       </material>
     </visual>
-    <!--<collision>
+    <collision>
       <origin xyz="0 0 0" rpy="0 1.5707963268 1.5707963268"/>
       <geometry>
         <mesh filename="package://minibot_description/meshes/shoulder_con_coll.dae"  scale="1 1 1"/>
       </geometry>
-    </collision>-->
+    </collision>
   </link>
   <link name="L_SHOULDER_ROLL_R" >
@@ -196,10 +196,10 @@
       </material>
     </visual>
-    <!--<collision>
+    <collision>
       <origin xyz="0 0 0" rpy="0 0 -1.5707963268" />
       <geometry>
         <mesh filename="package://minibot_description/meshes/upper_arm_coll.dae"  scale="1 1 1"/>
       </geometry>
-    </collision>-->
+    </collision>
   </link>
   <link name="L_ELBOW_R" >
@@ -220,10 +220,10 @@
       </material>
     </visual>
-    <!--<collision>
+    <collision>
       <origin xyz="0 0 0" rpy="0 1.5707963268 1.5707963268" />
       <geometry>
         <mesh filename="package://minibot_description/meshes/lower_arm_coll.dae"  scale="1 1 1"/>
       </geometry>
-    </collision>-->
+    </collision>
   </link>
   <link name="L_HIP_YAW_L" >
@@ -244,10 +244,10 @@
       </material>
     </visual>
-    <!--<collision>
+    <collision>
       <origin xyz="0 0 0" rpy="1.5707963268 0 0" />
       <geometry>
         <mesh filename="package://minibot_description/meshes/yaw_con_coll.dae"  scale="1 1 1"/>
       </geometry>
-    </collision>-->
+    </collision>
   </link>
   <link name="L_HIP_ROLL_L" >
@@ -269,10 +269,10 @@
       </material>
     </visual>
-    <!--<collision>
+    <collision>
       <origin xyz="0 0 -0.025" rpy="0 3.14 0" />
       <geometry>
         <mesh filename="package://minibot_description/meshes/hip_roll_coll.dae"  scale="1 1 1"/>
       </geometry>
-    </collision>-->
+    </collision>
   </link>
   <link name="L_HIP_PITCH_L" >
@@ -294,10 +294,10 @@
       </material>
     </visual>
-    <!--<collision>
+    <collision>
       <origin xyz="0 0 0" rpy="1.5707963268 1.5707963268 0" />
       <geometry>
         <mesh filename="package://minibot_description/meshes/upper_leg_coll.dae"  scale="1 1 1"/>
       </geometry>
-    </collision>-->
+    </collision>
   </link>
   <link name="L_KNEE_L" >
@@ -319,10 +319,10 @@
       </material>
     </visual>
-    <!--<collision>
+    <collision>
       <origin xyz="0 0 0" rpy="1.5707963268 1.5707963268 0" />
       <geometry>
         <mesh filename="package://minibot_description/meshes/lower_leg_coll.dae"  scale="1 1 1"/>
       </geometry>
-    </collision>-->
+    </collision>
   </link>
   <link name="L_ANKLE_PITCH_L" >
@@ -344,10 +344,10 @@
       </material>
     </visual>
-    <!--<collision>
+    <collision>
       <origin xyz="0 0 0" rpy="3.14 -1.5707963268 1.5707963268" />
       <geometry>
         <mesh filename="package://minibot_description/meshes/ankle_roll_coll.dae"  scale="1 1 1"/>
       </geometry>
-    </collision>-->
+    </collision>
   </link>
   <link name="L_ANKLE_ROLL_L" >
@@ -392,10 +392,10 @@
       </material>
     </visual>
-    <!--<collision>
+    <collision>
       <origin xyz="0 0 0" rpy="1.5707963268 0 0" />
       <geometry>
         <mesh filename="package://minibot_description/meshes/yaw_con_coll.dae"  scale="1 1 1"/>
       </geometry>
-    </collision>-->
+    </collision>
   </link>
   <link name="L_HIP_ROLL_R" >
@@ -417,10 +417,10 @@
       </material>
     </visual>
-    <!--<collision>
+    <collision>
       <origin xyz="0 0 -0.025" rpy="0 3.14 0" />
       <geometry>
         <mesh filename="package://minibot_description/meshes/hip_roll_coll.dae"  scale="1 1 1"/>
       </geometry>
-    </collision>-->
+    </collision>
   </link>
   <link name="L_HIP_PITCH_R" >
@@ -442,10 +442,10 @@
       </material>
     </visual>
-    <!--<collision>
+    <collision>
       <origin xyz="0 0 0" rpy="1.5707963268 -1.5707963268 0" />
       <geometry>
         <mesh filename="package://minibot_description/meshes/upper_leg_coll.dae"  scale="1 1 1"/>
       </geometry>
-    </collision>-->
+    </collision>
   </link>
   <link name="L_KNEE_R" >
@@ -467,10 +467,10 @@
       </material>
     </visual>
-    <!--<collision>
+    <collision>
       <origin xyz="0 0 0" rpy="1.5707963268 -1.5707963268 0" />
       <geometry>
         <mesh filename="package://minibot_description/meshes/lower_leg_coll.dae"  scale="1 1 1"/>
       </geometry>
-    </collision>-->
+    </collision>
   </link>
   <link name="L_ANKLE_PITCH_R" >
@@ -492,10 +492,10 @@
       </material>
     </visual>
-    <!--<collision>
+    <collision>
       <origin xyz="0 0 0" rpy="0 1.5707963268 1.5707963268" />
       <geometry>
         <mesh filename="package://minibot_description/meshes/ankle_roll_coll.dae"  scale="1 1 1"/>
       </geometry>
-    </collision>-->
+    </collision>
   </link>
   <link name="L_ANKLE_ROLL_R" >
@@ -1006,5 +1006,5 @@
     </plugin>
   </gazebo>
-  <!--<gazebo reference="L_CAMERA">
+  <gazebo reference="L_CAMERA">
         <sensor name='camera' type='camera'>
           <pose>-0.050000 -0.010000 0.000000 -1.5708 0.000000 -3.141592</pose>
@@ -1038,5 +1038,5 @@
           </plugin>
       </sensor>
-  </gazebo> -->
+  </gazebo>
       <gazebo>
         <plugin filename="libhector_gazebo_ros_imu.so" name="gazebo_ros_imu">
