Commit message: improved minibot simulation

File: minibot_description/urdf/minibot.urdf (robot description, URDF)
Before this commit: robot Minibot, 30 links, 29 joints
Joints:
- joint HeadPan: limit lower=-2.1816615649875 upper=2.1816615649875 effort=2.5 velocity=5.6548668 -> lower=-2.1816615649875 upper=2.1816615649875 effort=5.0 velocity=5.6548668
- joint HeadTilt: limit lower=-1.5707963267910001 upper=0 effort=2.5 velocity=5.6548668 -> lower=-1.5707963267910001 upper=0 effort=5.0 velocity=5.6548668
- joint LAnklePitch: limit lower=-1.6406094968706 upper=1.2391837689129 effort=8.4 velocity=4.712388975 -> lower=-1.6406094968706 upper=1.2391837689129 effort=16.8 velocity=4.712388975
- joint LAnkleRoll: limit lower=-1.4660765716716 upper=1.4660765716716 effort=6.0 velocity=6.597344565 -> lower=-1.4660765716716 upper=1.4660765716716 effort=12.0 velocity=6.597344565
- joint LElbow: limit lower=-1.1344640137935 upper=1.5707963267910001 effort=2.5 velocity=5.6548668 -> lower=-1.1344640137935 upper=1.5707963267910001 effort=5.0 velocity=5.6548668
- joint LHipPitch: limit lower=-0.48869219055720003 upper=1.919862177189 effort=8.4 velocity=4.712388975 -> lower=-0.48869219055720003 upper=1.919862177189 effort=16.8 velocity=4.712388975
- joint LHipRoll: limit lower=-1.0122909661542001 upper=0.7853981633955001 effort=6.0 velocity=6.597344565 -> lower=-1.0122909661542001 upper=0.7853981633955001 effort=12.0 velocity=6.597344565
- joint LHipYaw: limit lower=-0.9250245035547 upper=0.9250245035547 effort=2.5 velocity=5.6548668 -> lower=-0.9250245035547 upper=0.9250245035547 effort=5.0 velocity=5.6548668
- joint LKnee: limit lower=-2.268928027587 upper=0 effort=8.4 velocity=4.712388975 -> lower=-2.268928027587 upper=0 effort=16.8 velocity=4.712388975
- joint LShoulderPitch: limit lower=-3.1415926535820002 upper=3.1415926535820002 effort=6.0 velocity=6.597344565 -> lower=-3.1415926535820002 upper=3.1415926535820002 effort=12.0 velocity=6.597344565
- joint LShoulderRoll: limit lower=-2.3561944901865 upper=0.7853981633955001 effort=2.5 velocity=5.648668 -> lower=-2.3561944901865 upper=0.7853981633955001 effort=5.0 velocity=5.648668
- joint RAnklePitch: limit lower=-1.2391837689129 upper=1.6406094968706 effort=8.4 velocity=4.712388975 -> lower=-1.2391837689129 upper=1.6406094968706 effort=16.8 velocity=4.712388975
- joint RAnkleRoll: limit lower=-1.4660765716716 upper=1.4660765716716 effort=6.0 velocity=6.597344565 -> lower=-1.4660765716716 upper=1.4660765716716 effort=12.0 velocity=6.597344565
- joint RElbow: limit lower=-1.635 upper=1.5707963267910001 effort=2.5 velocity=5.6548668 -> lower=-1.635 upper=1.5707963267910001 effort=5.0 velocity=5.6548668
- joint RHipPitch: limit lower=-1.919862177189 upper=0.48869219055720003 effort=8.4 velocity=4.712388975 -> lower=-1.919862177189 upper=0.48869219055720003 effort=16.8 velocity=4.712388975
- joint RHipRoll: limit lower=-1.0122909661542001 upper=0.7853981633955001 effort=6.0 velocity=6.597344565 -> lower=-1.0122909661542001 upper=0.7853981633955001 effort=12.0 velocity=6.597344565
- joint RHipYaw: limit lower=-0.9250245035547 upper=0.9250245035547 effort=2.5 velocity=5.6548668 -> lower=-0.9250245035547 upper=0.9250245035547 effort=5.0 velocity=5.6548668
- joint RKnee: limit lower=0 upper=2.268928027587 effort=8.4 velocity=4.712388975 -> lower=0 upper=2.268928027587 effort=16.8 velocity=4.712388975
- joint RShoulderPitch: limit lower=-3.1415926535820002 upper=3.1415926535820002 effort=6.0 velocity=6.597344565 -> lower=-3.1415926535820002 upper=3.1415926535820002 effort=12.0 velocity=6.597344565
- joint RShoulderRoll: limit lower=-0.7853981633955001 upper=2.3561944901865 effort=2.5 velocity=5.648668 -> lower=-0.7853981633955001 upper=2.3561944901865 effort=5.0 velocity=5.648668

File: minibot_description/urdf/minibot.urdf.xacro (robot description, xacro)
@@ -6,4 +6,5 @@
 <xacro:property name="d" value="0" /> <!-- damping -->
 <xacro:property name="f" value="0" /> <!-- friction -->
+<xacro:property name="pos_or_eff" value="1" /> <!-- position (0) or effort(1) joint interfaces -->
 <link name="base_link"/>
   <joint name="base_link_to_body" type="fixed">
@@ -717,9 +718,19 @@
     <type>transmission_interface/SimpleTransmission</type>
     <joint name="HeadPan">
-        <hardwareInterface>EffortJointInterface</hardwareInterface>
+    <xacro:if value="${pos_or_eff == 0}">
+        <hardwareInterface>hardware_interface/PositionJointInterface</hardwareInterface>
+    </xacro:if>
+    <xacro:if value="${pos_or_eff == 1}">
+        <hardwareInterface>hardware_interface/EffortJointInterface</hardwareInterface>
+    </xacro:if>
     </joint>
     <actuator name="HeadPanMotor">
-      <hardwareInterface>EffortJointInterface</hardwareInterface>
-      <mechanicalReduction>1</mechanicalReduction>
+        <xacro:if value="${pos_or_eff == 0}">
+            <hardwareInterface>hardware_interface/PositionJointInterface</hardwareInterface>
+        </xacro:if>
+        <xacro:if value="${pos_or_eff == 1}">
+            <hardwareInterface>hardware_interface/EffortJointInterface</hardwareInterface>
+        </xacro:if>
+        <mechanicalReduction>1</mechanicalReduction>
     </actuator>
   </transmission>
@@ -727,8 +738,18 @@
     <type>transmission_interface/SimpleTransmission</type>
     <joint name="HeadTilt">
-        <hardwareInterface>EffortJointInterface</hardwareInterface>
+        <xacro:if value="${pos_or_eff == 0}">
+            <hardwareInterface>hardware_interface/PositionJointInterface</hardwareInterface>
+        </xacro:if>
+        <xacro:if value="${pos_or_eff == 1}">
+            <hardwareInterface>hardware_interface/EffortJointInterface</hardwareInterface>
+        </xacro:if>
     </joint>
     <actuator name="HeadTiltMotor">
-      <hardwareInterface>EffortJointInterface</hardwareInterface>
+        <xacro:if value="${pos_or_eff == 0}">
+            <hardwareInterface>hardware_interface/PositionJointInterface</hardwareInterface>
+        </xacro:if>
+        <xacro:if value="${pos_or_eff == 1}">
+            <hardwareInterface>hardware_interface/EffortJointInterface</hardwareInterface>
+        </xacro:if>
       <mechanicalReduction>1</mechanicalReduction>
     </actuator>
@@ -737,8 +758,18 @@
     <type>transmission_interface/SimpleTransmission</type>
     <joint name="LShoulderPitch">
-        <hardwareInterface>EffortJointInterface</hardwareInterface>
+        <xacro:if value="${pos_or_eff == 0}">
+            <hardwareInterface>hardware_interface/PositionJointInterface</hardwareInterface>
+        </xacro:if>
+        <xacro:if value="${pos_or_eff == 1}">
+            <hardwareInterface>hardware_interface/EffortJointInterface</hardwareInterface>
+        </xacro:if>
     </joint>
     <actuator name="LShoulderPitchMotor">
-      <hardwareInterface>EffortJointInterface</hardwareInterface>
+        <xacro:if value="${pos_or_eff == 0}">
+            <hardwareInterface>hardware_interface/PositionJointInterface</hardwareInterface>
+        </xacro:if>
+        <xacro:if value="${pos_or_eff == 1}">
+            <hardwareInterface>hardware_interface/EffortJointInterface</hardwareInterface>
+        </xacro:if>
       <mechanicalReduction>1</mechanicalReduction>
     </actuator>
@@ -747,8 +778,18 @@
     <type>transmission_interface/SimpleTransmission</type>
     <joint name="LShoulderRoll">
-        <hardwareInterface>EffortJointInterface</hardwareInterface>
+        <xacro:if value="${pos_or_eff == 0}">
+            <hardwareInterface>hardware_interface/PositionJointInterface</hardwareInterface>
+        </xacro:if>
+        <xacro:if value="${pos_or_eff == 1}">
+            <hardwareInterface>hardware_interface/EffortJointInterface</hardwareInterface>
+        </xacro:if>
     </joint>
     <actuator name="LShoulderRollTransmission">
-      <hardwareInterface>EffortJointInterface</hardwareInterface>
+        <xacro:if value="${pos_or_eff == 0}">
+            <hardwareInterface>hardware_interface/PositionJointInterface</hardwareInterface>
+        </xacro:if>
+        <xacro:if value="${pos_or_eff == 1}">
+            <hardwareInterface>hardware_interface/EffortJointInterface</hardwareInterface>
+        </xacro:if>
       <mechanicalReduction>1</mechanicalReduction>
     </actuator>
@@ -757,8 +798,18 @@
     <type>transmission_interface/SimpleTransmission</type>
     <joint name="LElbow">
-        <hardwareInterface>EffortJointInterface</hardwareInterface>
+        <xacro:if value="${pos_or_eff == 0}">
+            <hardwareInterface>hardware_interface/PositionJointInterface</hardwareInterface>
+        </xacro:if>
+        <xacro:if value="${pos_or_eff == 1}">
+            <hardwareInterface>hardware_interface/EffortJointInterface</hardwareInterface>
+        </xacro:if>
     </joint>
     <actuator name="LElbowMotor">
-      <hardwareInterface>EffortJointInterface</hardwareInterface>
+        <xacro:if value="${pos_or_eff == 0}">
+            <hardwareInterface>hardware_interface/PositionJointInterface</hardwareInterface>
+        </xacro:if>
+        <xacro:if value="${pos_or_eff == 1}">
+            <hardwareInterface>hardware_interface/EffortJointInterface</hardwareInterface>
+        </xacro:if>
       <mechanicalReduction>1</mechanicalReduction>
     </actuator>
@@ -767,8 +818,18 @@
     <type>transmission_interface/SimpleTransmission</type>
     <joint name="RShoulderPitch">
-        <hardwareInterface>EffortJointInterface</hardwareInterface>
+        <xacro:if value="${pos_or_eff == 0}">
+            <hardwareInterface>hardware_interface/PositionJointInterface</hardwareInterface>
+        </xacro:if>
+        <xacro:if value="${pos_or_eff == 1}">
+            <hardwareInterface>hardware_interface/EffortJointInterface</hardwareInterface>
+        </xacro:if>
     </joint>
     <actuator name="RShoulderPitchMotor">
-      <hardwareInterface>EffortJointInterface</hardwareInterface>
+        <xacro:if value="${pos_or_eff == 0}">
+            <hardwareInterface>hardware_interface/PositionJointInterface</hardwareInterface>
+        </xacro:if>
+        <xacro:if value="${pos_or_eff == 1}">
+            <hardwareInterface>hardware_interface/EffortJointInterface</hardwareInterface>
+        </xacro:if>
       <mechanicalReduction>1</mechanicalReduction>
     </actuator>
@@ -777,8 +838,18 @@
     <type>transmission_interface/SimpleTransmission</type>
     <joint name="RShoulderRoll">
-        <hardwareInterface>EffortJointInterface</hardwareInterface>
+        <xacro:if value="${pos_or_eff == 0}">
+            <hardwareInterface>hardware_interface/PositionJointInterface</hardwareInterface>
+        </xacro:if>
+        <xacro:if value="${pos_or_eff == 1}">
+            <hardwareInterface>hardware_interface/EffortJointInterface</hardwareInterface>
+        </xacro:if>
     </joint>
     <actuator name="RShoulderRollMotor">
-      <hardwareInterface>EffortJointInterface</hardwareInterface>
+        <xacro:if value="${pos_or_eff == 0}">
+            <hardwareInterface>hardware_interface/PositionJointInterface</hardwareInterface>
+        </xacro:if>
+        <xacro:if value="${pos_or_eff == 1}">
+            <hardwareInterface>hardware_interface/EffortJointInterface</hardwareInterface>
+        </xacro:if>
       <mechanicalReduction>1</mechanicalReduction>
     </actuator>
@@ -787,8 +858,18 @@
     <type>transmission_interface/SimpleTransmission</type>
     <joint name="RElbow">
-        <hardwareInterface>EffortJointInterface</hardwareInterface>
+        <xacro:if value="${pos_or_eff == 0}">
+            <hardwareInterface>hardware_interface/PositionJointInterface</hardwareInterface>
+        </xacro:if>
+        <xacro:if value="${pos_or_eff == 1}">
+            <hardwareInterface>hardware_interface/EffortJointInterface</hardwareInterface>
+        </xacro:if>
     </joint>
     <actuator name="RElbowMotor">
-      <hardwareInterface>EffortJointInterface</hardwareInterface>
+        <xacro:if value="${pos_or_eff == 0}">
+            <hardwareInterface>hardware_interface/PositionJointInterface</hardwareInterface>
+        </xacro:if>
+        <xacro:if value="${pos_or_eff == 1}">
+            <hardwareInterface>hardware_interface/EffortJointInterface</hardwareInterface>
+        </xacro:if>
       <mechanicalReduction>1</mechanicalReduction>
     </actuator>
@@ -797,8 +878,18 @@
     <type>transmission_interface/SimpleTransmission</type>
     <joint name="LHipYaw">
-        <hardwareInterface>EffortJointInterface</hardwareInterface>
+        <xacro:if value="${pos_or_eff == 0}">
+            <hardwareInterface>hardware_interface/PositionJointInterface</hardwareInterface>
+        </xacro:if>
+        <xacro:if value="${pos_or_eff == 1}">
+            <hardwareInterface>hardware_interface/EffortJointInterface</hardwareInterface>
+        </xacro:if>
     </joint>
     <actuator name="LHipYawMotor">
-      <hardwareInterface>EffortJointInterface</hardwareInterface>
+        <xacro:if value="${pos_or_eff == 0}">
+            <hardwareInterface>hardware_interface/PositionJointInterface</hardwareInterface>
+        </xacro:if>
+        <xacro:if value="${pos_or_eff == 1}">
+            <hardwareInterface>hardware_interface/EffortJointInterface</hardwareInterface>
+        </xacro:if>
       <mechanicalReduction>1</mechanicalReduction>
     </actuator>
@@ -807,8 +898,18 @@
     <type>transmission_interface/SimpleTransmission</type>
     <joint name="LHipRoll">
-        <hardwareInterface>EffortJointInterface</hardwareInterface>
+        <xacro:if value="${pos_or_eff == 0}">
+            <hardwareInterface>hardware_interface/PositionJointInterface</hardwareInterface>
+        </xacro:if>
+        <xacro:if value="${pos_or_eff == 1}">
+            <hardwareInterface>hardware_interface/EffortJointInterface</hardwareInterface>
+        </xacro:if>
     </joint>
     <actuator name="LHipRollMotor">
-      <hardwareInterface>EffortJointInterface</hardwareInterface>
+        <xacro:if value="${pos_or_eff == 0}">
+            <hardwareInterface>hardware_interface/PositionJointInterface</hardwareInterface>
+        </xacro:if>
+        <xacro:if value="${pos_or_eff == 1}">
+            <hardwareInterface>hardware_interface/EffortJointInterface</hardwareInterface>
+        </xacro:if>
       <mechanicalReduction>1</mechanicalReduction>
     </actuator>
@@ -817,8 +918,18 @@
     <type>transmission_interface/SimpleTransmission</type>
     <joint name="LHipPitch">
-        <hardwareInterface>EffortJointInterface</hardwareInterface>
+        <xacro:if value="${pos_or_eff == 0}">
+            <hardwareInterface>hardware_interface/PositionJointInterface</hardwareInterface>
+        </xacro:if>
+        <xacro:if value="${pos_or_eff == 1}">
+            <hardwareInterface>hardware_interface/EffortJointInterface</hardwareInterface>
+        </xacro:if>
     </joint>
     <actuator name="LHipPitchMotor">
-      <hardwareInterface>EffortJointInterface</hardwareInterface>
+        <xacro:if value="${pos_or_eff == 0}">
+            <hardwareInterface>hardware_interface/PositionJointInterface</hardwareInterface>
+        </xacro:if>
+        <xacro:if value="${pos_or_eff == 1}">
+            <hardwareInterface>hardware_interface/EffortJointInterface</hardwareInterface>
+        </xacro:if>
       <mechanicalReduction>1</mechanicalReduction>
     </actuator>
@@ -827,8 +938,18 @@
     <type>transmission_interface/SimpleTransmission</type>
     <joint name="LKnee">
-        <hardwareInterface>EffortJointInterface</hardwareInterface>
+        <xacro:if value="${pos_or_eff == 0}">
+            <hardwareInterface>hardware_interface/PositionJointInterface</hardwareInterface>
+        </xacro:if>
+        <xacro:if value="${pos_or_eff == 1}">
+            <hardwareInterface>hardware_interface/EffortJointInterface</hardwareInterface>
+        </xacro:if>
     </joint>
     <actuator name="LKneeMotor">
-      <hardwareInterface>EffortJointInterface</hardwareInterface>
+        <xacro:if value="${pos_or_eff == 0}">
+            <hardwareInterface>hardware_interface/PositionJointInterface</hardwareInterface>
+        </xacro:if>
+        <xacro:if value="${pos_or_eff == 1}">
+            <hardwareInterface>hardware_interface/EffortJointInterface</hardwareInterface>
+        </xacro:if>
       <mechanicalReduction>1</mechanicalReduction>
     </actuator>
@@ -837,8 +958,18 @@
     <type>transmission_interface/SimpleTransmission</type>
     <joint name="LAnklePitch">
-        <hardwareInterface>EffortJointInterface</hardwareInterface>
+        <xacro:if value="${pos_or_eff == 0}">
+            <hardwareInterface>hardware_interface/PositionJointInterface</hardwareInterface>
+        </xacro:if>
+        <xacro:if value="${pos_or_eff == 1}">
+            <hardwareInterface>hardware_interface/EffortJointInterface</hardwareInterface>
+        </xacro:if>
     </joint>
     <actuator name="LAnklePitchMotor">
-      <hardwareInterface>EffortJointInterface</hardwareInterface>
+        <xacro:if value="${pos_or_eff == 0}">
+            <hardwareInterface>hardware_interface/PositionJointInterface</hardwareInterface>
+        </xacro:if>
+        <xacro:if value="${pos_or_eff == 1}">
+            <hardwareInterface>hardware_interface/EffortJointInterface</hardwareInterface>
+        </xacro:if>
       <mechanicalReduction>1</mechanicalReduction>
     </actuator>
@@ -847,8 +978,18 @@
     <type>transmission_interface/SimpleTransmission</type>
     <joint name="LAnkleRoll">
-        <hardwareInterface>EffortJointInterface</hardwareInterface>
+        <xacro:if value="${pos_or_eff == 0}">
+            <hardwareInterface>hardware_interface/PositionJointInterface</hardwareInterface>
+        </xacro:if>
+        <xacro:if value="${pos_or_eff == 1}">
+            <hardwareInterface>hardware_interface/EffortJointInterface</hardwareInterface>
+        </xacro:if>
     </joint>
     <actuator name="LAnkleRollMotor">
-      <hardwareInterface>EffortJointInterface</hardwareInterface>
+        <xacro:if value="${pos_or_eff == 0}">
+            <hardwareInterface>hardware_interface/PositionJointInterface</hardwareInterface>
+        </xacro:if>
+        <xacro:if value="${pos_or_eff == 1}">
+            <hardwareInterface>hardware_interface/EffortJointInterface</hardwareInterface>
+        </xacro:if>
       <mechanicalReduction>1</mechanicalReduction>
     </actuator>
@@ -857,8 +998,18 @@
     <type>transmission_interface/SimpleTransmission</type>
     <joint name="RHipYaw">
-        <hardwareInterface>EffortJointInterface</hardwareInterface>
+        <xacro:if value="${pos_or_eff == 0}">
+            <hardwareInterface>hardware_interface/PositionJointInterface</hardwareInterface>
+        </xacro:if>
+        <xacro:if value="${pos_or_eff == 1}">
+            <hardwareInterface>hardware_interface/EffortJointInterface</hardwareInterface>
+        </xacro:if>
     </joint>
     <actuator name="RHipYawMotor">
-      <hardwareInterface>EffortJointInterface</hardwareInterface>
+        <xacro:if value="${pos_or_eff == 0}">
+            <hardwareInterface>hardware_interface/PositionJointInterface</hardwareInterface>
+        </xacro:if>
+        <xacro:if value="${pos_or_eff == 1}">
+            <hardwareInterface>hardware_interface/EffortJointInterface</hardwareInterface>
+        </xacro:if>
       <mechanicalReduction>1</mechanicalReduction>
     </actuator>
@@ -867,8 +1018,18 @@
     <type>transmission_interface/SimpleTransmission</type>
     <joint name="RHipRoll">
-        <hardwareInterface>EffortJointInterface</hardwareInterface>
+        <xacro:if value="${pos_or_eff == 0}">
+            <hardwareInterface>hardware_interface/PositionJointInterface</hardwareInterface>
+        </xacro:if>
+        <xacro:if value="${pos_or_eff == 1}">
+            <hardwareInterface>hardware_interface/EffortJointInterface</hardwareInterface>
+        </xacro:if>
     </joint>
     <actuator name="RHipRollMotor">
-      <hardwareInterface>EffortJointInterface</hardwareInterface>
+        <xacro:if value="${pos_or_eff == 0}">
+            <hardwareInterface>hardware_interface/PositionJointInterface</hardwareInterface>
+        </xacro:if>
+        <xacro:if value="${pos_or_eff == 1}">
+            <hardwareInterface>hardware_interface/EffortJointInterface</hardwareInterface>
+        </xacro:if>
       <mechanicalReduction>1</mechanicalReduction>
     </actuator>
@@ -877,8 +1038,18 @@
     <type>transmission_interface/SimpleTransmission</type>
     <joint name="RHipPitch">
-        <hardwareInterface>EffortJointInterface</hardwareInterface>
+        <xacro:if value="${pos_or_eff == 0}">
+            <hardwareInterface>hardware_interface/PositionJointInterface</hardwareInterface>
+        </xacro:if>
+        <xacro:if value="${pos_or_eff == 1}">
+            <hardwareInterface>hardware_interface/EffortJointInterface</hardwareInterface>
+        </xacro:if>
     </joint>
     <actuator name="RHipPitchMotor">
-      <hardwareInterface>EffortJointInterface</hardwareInterface>
+        <xacro:if value="${pos_or_eff == 0}">
+            <hardwareInterface>hardware_interface/PositionJointInterface</hardwareInterface>
+        </xacro:if>
+        <xacro:if value="${pos_or_eff == 1}">
+            <hardwareInterface>hardware_interface/EffortJointInterface</hardwareInterface>
+        </xacro:if>
       <mechanicalReduction>1</mechanicalReduction>
     </actuator>
@@ -887,8 +1058,18 @@
     <type>transmission_interface/SimpleTransmission</type>
     <joint name="RKnee">
-        <hardwareInterface>EffortJointInterface</hardwareInterface>
+        <xacro:if value="${pos_or_eff == 0}">
+            <hardwareInterface>hardware_interface/PositionJointInterface</hardwareInterface>
+        </xacro:if>
+        <xacro:if value="${pos_or_eff == 1}">
+            <hardwareInterface>hardware_interface/EffortJointInterface</hardwareInterface>
+        </xacro:if>
     </joint>
     <actuator name="RKneeMotor">
-      <hardwareInterface>EffortJointInterface</hardwareInterface>
+        <xacro:if value="${pos_or_eff == 0}">
+            <hardwareInterface>hardware_interface/PositionJointInterface</hardwareInterface>
+        </xacro:if>
+        <xacro:if value="${pos_or_eff == 1}">
+            <hardwareInterface>hardware_interface/EffortJointInterface</hardwareInterface>
+        </xacro:if>
       <mechanicalReduction>1</mechanicalReduction>
     </actuator>
@@ -897,8 +1078,18 @@
     <type>transmission_interface/SimpleTransmission</type>
     <joint name="RAnklePitch">
-        <hardwareInterface>EffortJointInterface</hardwareInterface>
+        <xacro:if value="${pos_or_eff == 0}">
+            <hardwareInterface>hardware_interface/PositionJointInterface</hardwareInterface>
+        </xacro:if>
+        <xacro:if value="${pos_or_eff == 1}">
+            <hardwareInterface>hardware_interface/EffortJointInterface</hardwareInterface>
+        </xacro:if>
     </joint>
     <actuator name="RAnklePitchMotor">
-      <hardwareInterface>EffortJointInterface</hardwareInterface>
+        <xacro:if value="${pos_or_eff == 0}">
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