Commit message: improving simulator experience

File: minibot_description/urdf/minibot.urdf (robot description, URDF)
Before this commit: robot Minibot, 30 links, 29 joints
Joints:
- joint HeadPan: limit lower=-2.1816615649875 upper=2.1816615649875 effort=5.0 velocity=5.6548668 -> lower=-2.1816615649875 upper=2.1816615649875 effort=2.5 velocity=5.6548668
- joint HeadTilt: limit lower=-1.5707963267910001 upper=0 effort=5.0 velocity=5.6548668 -> lower=-1.5707963267910001 upper=0 effort=2.5 velocity=5.6548668
- joint LAnklePitch: limit lower=-1.6406094968706 upper=1.2391837689129 effort=16.8 velocity=4.712388975 -> lower=-1.6406094968706 upper=1.2391837689129 effort=8.4 velocity=4.712388975
- joint LAnkleRoll: limit lower=-1.4660765716716 upper=1.4660765716716 effort=12.0 velocity=6.597344565 -> lower=-1.4660765716716 upper=1.4660765716716 effort=6.0 velocity=6.597344565
- joint LElbow: limit lower=-1.1344640137935 upper=1.5707963267910001 effort=5.0 velocity=5.6548668 -> lower=-1.1344640137935 upper=1.5707963267910001 effort=2.5 velocity=5.6548668
- joint LHipPitch: limit lower=-0.48869219055720003 upper=1.919862177189 effort=16.8 velocity=4.712388975 -> lower=-0.48869219055720003 upper=1.919862177189 effort=8.4 velocity=4.712388975
- joint LHipRoll: limit lower=-1.0122909661542001 upper=0.7853981633955001 effort=12.0 velocity=6.597344565 -> lower=-1.0122909661542001 upper=0.7853981633955001 effort=6.0 velocity=6.597344565
- joint LHipYaw: limit lower=-0.9250245035547 upper=0.9250245035547 effort=5.0 velocity=5.6548668 -> lower=-0.9250245035547 upper=0.9250245035547 effort=2.5 velocity=5.6548668
- joint LKnee: limit lower=-2.268928027587 upper=0 effort=16.8 velocity=4.712388975 -> lower=-2.268928027587 upper=0 effort=8.4 velocity=4.712388975
- joint LShoulderPitch: limit lower=-3.1415926535820002 upper=3.1415926535820002 effort=12.0 velocity=6.597344565 -> lower=-3.1415926535820002 upper=3.1415926535820002 effort=6.0 velocity=6.597344565
- joint LShoulderRoll: limit lower=-2.3561944901865 upper=0.7853981633955001 effort=5.0 velocity=5.648668 -> lower=-2.3561944901865 upper=0.7853981633955001 effort=2.5 velocity=5.648668
- joint RAnklePitch: limit lower=-1.2391837689129 upper=1.6406094968706 effort=16.8 velocity=4.712388975 -> lower=-1.2391837689129 upper=1.6406094968706 effort=8.4 velocity=4.712388975
- joint RAnkleRoll: limit lower=-1.4660765716716 upper=1.4660765716716 effort=12.0 velocity=6.597344565 -> lower=-1.4660765716716 upper=1.4660765716716 effort=6.0 velocity=6.597344565
- joint RElbow: limit lower=-1.635 upper=1.5707963267910001 effort=5.0 velocity=5.6548668 -> lower=-1.635 upper=1.5707963267910001 effort=2.5 velocity=5.6548668
- joint RHipPitch: limit lower=-1.919862177189 upper=0.48869219055720003 effort=16.8 velocity=4.712388975 -> lower=-1.919862177189 upper=0.48869219055720003 effort=8.4 velocity=4.712388975
- joint RHipRoll: limit lower=-1.0122909661542001 upper=0.7853981633955001 effort=12.0 velocity=6.597344565 -> lower=-1.0122909661542001 upper=0.7853981633955001 effort=6.0 velocity=6.597344565
- joint RHipYaw: limit lower=-0.9250245035547 upper=0.9250245035547 effort=5.0 velocity=5.6548668 -> lower=-0.9250245035547 upper=0.9250245035547 effort=2.5 velocity=5.6548668
- joint RKnee: limit lower=0 upper=2.268928027587 effort=16.8 velocity=4.712388975 -> lower=0 upper=2.268928027587 effort=8.4 velocity=4.712388975
- joint RShoulderPitch: limit lower=-3.1415926535820002 upper=3.1415926535820002 effort=12.0 velocity=6.597344565 -> lower=-3.1415926535820002 upper=3.1415926535820002 effort=6.0 velocity=6.597344565
- joint RShoulderRoll: limit lower=-0.7853981633955001 upper=2.3561944901865 effort=5.0 velocity=5.648668 -> lower=-0.7853981633955001 upper=2.3561944901865 effort=2.5 velocity=5.648668

Commit message: URDF Motorwinkel korrigiert

File: minibot_description/urdf/minibot.urdf (robot description, URDF)
Before this commit: robot Minibot, 30 links, 29 joints
Joints:
- joint LHipRoll: axis 0 0 -1 -> 0 0 1

File: minibot_description/urdf/minibot.urdf.xacro (robot description, xacro)
@@ -622,5 +622,5 @@
     <child link="L_HIP_ROLL_L"/>
     <origin xyz="-0.025 0 0.038444" rpy="-1.5707963 0 1.5707963" />
-    <axis xyz="0 0 -1" />
+    <axis xyz="0 0 1" />
     <limit effort="${tofa*6.0}" velocity="6.597344565" lower="-1.0122909661542001" upper="0.7853981633955001" />
   <dynamics damping="${d}" friction="0.0"/> </joint>

Commit message: removed mass from minibot head to counter simulation errors

File: minibot_description/urdf/minibot.urdf (robot description, URDF)
Before this commit: robot Minibot, 30 links, 29 joints
Links:
- link L_HEAD_PAN: mass 0.012 -> 0.001
- link L_HEAD_TILT: mass 0.139 -> 0.001

File: minibot_description/urdf/minibot.urdf.xacro (robot description, xacro)
@@ -40,7 +40,9 @@
     <inertial>
       <origin xyz="0.000002 -0.001022 0.008994"/>
-      <mass value="0.012"/>
+            <mass value="0.001"/>
+      <inertia ixx="0"  ixy="0"  ixz="0" iyy="0" iyz="0" izz="0" />
+      <!--<mass value="0.012"/>-->
       <!--<inertia ixx="0.000001769"  ixy="0.0"  ixz="0.0" iyy="0.000004625" iyz="-0.000000082" izz="0.000005125" />-->
-      <inertia ixx="${insu*0.1+infa*0.000001769}"  ixy="0.0"  ixz="0" iyy="${insu*0.1+infa*0.000004625}" iyz="0.0" izz="${insu*0.1+infa*0.000005125}" />
+      <!--<inertia ixx="${insu*0.1+infa*0.000001769}"  ixy="0.0"  ixz="0" iyy="${insu*0.1+infa*0.000004625}" iyz="0.0" izz="${insu*0.1+infa*0.000005125}" />-->
       <!--<inertia ixx="0.001"  ixy="0.001"  ixz="0.001" iyy="0.001" iyz="0.001" izz="0.001" />-->
     </inertial>
@@ -64,6 +66,8 @@
     <inertial>
       <origin xyz="-0.000223 -0.028433 0.0" rpy="0 1.5707963268 0"/>
-      <mass value="0.139"/>
-      <inertia ixx="${insu*0.1+infa*0.000097954}"  ixy="0"  ixz="0" iyy="${insu*0.1+infa*0.000025415}" iyz="0" izz="${insu*0.1+infa*0.000107764}" />
+      <mass value="0.001"/>
+      <inertia ixx="0"  ixy="0"  ixz="0" iyy="0" iyz="0" izz="0" />
+      <!--<mass value="0.139"/>
+      <inertia ixx="${insu*0.1+infa*0.000097954}"  ixy="0"  ixz="0" iyy="${insu*0.1+infa*0.000025415}" iyz="0" izz="${insu*0.1+infa*0.000107764}" /> -->
       <!--<inertia ixx="0.001"  ixy="0.001"  ixz="0.001" iyy="0.001" iyz="0.001" izz="0.001" />-->
     </inertial>

Commit message: changed urdf for moveit quintic walk

File: minibot_description/urdf/minibot.urdf (robot description, URDF)
Before this commit: robot Minibot, 30 links, 29 joints
Links:
- removed link L_FOOT_BOTTOM_L
- removed link L_FOOT_BOTTOM_R
- removed link L_TORSO
- added link left_foot_sole_link
- added link right_foot_sole_link
- added link trunk_link, mass 1.423; collision mesh filename=package://minibot_description/meshes/torso_coll.dae scale=1 1 1; visual mesh filename=package://minibot_description/meshes/torso_low.dae scale=1 1 1
Joints:
- joint HeadPan: parent L_TORSO -> trunk_link
- joint LHipYaw: parent L_TORSO -> trunk_link
- joint LShoulderPitch: parent L_TORSO -> trunk_link
- joint RHipYaw: parent L_TORSO -> trunk_link
- joint RShoulderPitch: parent L_TORSO -> trunk_link
- joint base_link_to_body: child L_TORSO -> trunk_link
- joint j_LFootBottom: child L_FOOT_BOTTOM_L -> left_foot_sole_link
- joint j_LFootFront: parent L_FOOT_BOTTOM_L -> left_foot_sole_link
- joint j_RFootBottom: child L_FOOT_BOTTOM_R -> right_foot_sole_link
- joint j_RFootFront: parent L_FOOT_BOTTOM_R -> right_foot_sole_link
- joint j_imu: parent L_TORSO -> trunk_link

File: minibot_description/urdf/minibot.urdf.xacro (robot description, xacro)
@@ -10,8 +10,8 @@
   <joint name="base_link_to_body" type="fixed">
     <parent link="base_link"/>
-    <child link="L_TORSO"/>
+    <child link="trunk_link"/>
     <origin xyz="0 0 0.545" rpy="0 0 0" />
   </joint>
-  <link name="L_TORSO">
+  <link name="trunk_link">
     <inertial>
       <origin xyz="-0.025019 0.000832 -0.054364" rpy=" 1.5707963268 0 1.5707963268"/>
@@ -531,6 +531,6 @@
   <link name="L_Hand_L" />
   <link name="L_Hand_R" />
-  <link name="L_FOOT_BOTTOM_L" />
-  <link name="L_FOOT_BOTTOM_R" />
+  <link name="left_foot_sole_link" />
+  <link name="right_foot_sole_link" />
   <link name="L_FOOT_FRONT_L" />
   <link name="L_FOOT_FRONT_R" />
@@ -538,5 +538,5 @@
   </link>
   <joint name="j_imu" type="fixed">
-  <parent link="L_TORSO"/>
+  <parent link="trunk_link"/>
   <child link="L_IMU"/>
   <origin xyz="-0.03 0 -0.05" rpy="0 0 0" />
@@ -557,5 +557,5 @@
   <dynamics damping="${d}" friction="0.0"/> </joint>
   <joint name="HeadPan" type="revolute">
-    <parent link="L_TORSO"/>
+    <parent link="trunk_link"/>
     <child link="L_HEAD_PAN"/>
     <origin xyz="0 0 0.050593" rpy="0 0 1.5707963" />
@@ -564,5 +564,5 @@
   <dynamics damping="${d}" friction="0.0"/> </joint>
   <joint name="LShoulderPitch" type="revolute">
-    <parent link="L_TORSO"/>
+    <parent link="trunk_link"/>
     <child link="L_SHOULDER_PITCH_L"/>
     <origin xyz="0 0.08134 0" rpy="0 -1.5707963 -1.5707963" />
@@ -590,5 +590,5 @@
   </joint>
   <joint name="RShoulderPitch" type="revolute">
-    <parent link="L_TORSO"/>
+    <parent link="trunk_link"/>
     <child link="L_SHOULDER_PITCH_R"/>
     <origin xyz="0 -0.08134 0" rpy="0 1.5707963 -1.5707963" />
@@ -616,5 +616,5 @@
   </joint>
   <joint name="LHipYaw" type="revolute">
-    <parent link="L_TORSO"/>
+    <parent link="trunk_link"/>
     <child link="L_HIP_YAW_L"/>
     <origin xyz="-0.022 0.057775 -0.160593" rpy="0 3.14159 3.14159" />
@@ -659,14 +659,14 @@
   <joint name="j_LFootBottom" type="fixed">
    <parent link="L_ANKLE_ROLL_L"/>
-   <child link="L_FOOT_BOTTOM_L" />
+   <child link="left_foot_sole_link" />
    <origin xyz="-0.040444 0 0" rpy="3.14159 -1.5707963 0"/>
   </joint>
   <joint name="j_LFootFront" type="fixed">
-   <parent link="L_FOOT_BOTTOM_L"/>
+   <parent link="left_foot_sole_link"/>
    <child link="L_FOOT_FRONT_L" />
    <origin xyz="0.0849 0 0 "/>
   </joint>
   <joint name="RHipYaw" type="revolute">
-    <parent link="L_TORSO"/>
+    <parent link="trunk_link"/>
     <child link="L_HIP_YAW_R"/>
     <origin xyz="-0.022 -0.057775 -0.160593" rpy="0 3.14159 3.14159" />
@@ -711,9 +711,9 @@
   <joint name="j_RFootBottom" type="fixed">
    <parent link="L_ANKLE_ROLL_R"/>
-   <child link="L_FOOT_BOTTOM_R" />
+   <child link="right_foot_sole_link" />
    <origin xyz="0.040444 0 0" rpy="0 -1.5707963 0"/>
   </joint>
   <joint name="j_RFootFront" type="fixed">
-   <parent link="L_FOOT_BOTTOM_R"/>
+   <parent link="right_foot_sole_link"/>
    <child link="L_FOOT_FRONT_R" />
    <origin xyz="0.0849 0 0 "/>
@@ -1119,5 +1119,5 @@
     </actuator>
   </transmission>
-<gazebo reference="L_TORSO">
+<gazebo reference="trunk_link">
     <material>Gazebo/Grey</material>
   </gazebo>

Commit message: fixes for walking

File: minibot_description/urdf/minibot.urdf (robot description, URDF)
Before this commit: robot Minibot, 30 links, 29 joints
Links:
- removed link base_link
- added link torso_link, mass 1.423; collision mesh filename=package://minibot_description/meshes/torso_coll.dae scale=1 1 1; visual mesh filename=package://minibot_description/meshes/torso_low.dae scale=1 1 1
- link trunk_link: mass 1.423 -> None; geometry 
Joints:
- removed joint base_link_to_body
- added joint torso: type fixed, parent trunk_link, child torso_link, origin xyz=0.022 0 0.160593 rpy=0 0 0, axis 0 0 1
- joint HeadPan: parent trunk_link -> torso_link
- joint LAnkleRoll: origin xyz=0 0.0275 0 rpy=-1.5707963 0 0 -> xyz=0 0 0 rpy=-1.5707963 0 0
- joint LHipPitch: origin xyz=0 0 -0.025 rpy=1.5707963 0 1.5707963 -> xyz=0 0 0 rpy=1.5707963 0 1.5707963
- joint LHipRoll: origin xyz=-0.025 0 0.038444 rpy=-1.5707963 0 1.5707963 -> xyz=0 0 0.038444 rpy=-1.5707963 0 1.5707963
- joint LHipYaw: origin xyz=-0.022 0.057775 -0.160593 rpy=0 3.14159 3.14159 -> xyz=0 0.057775 0 rpy=0 3.14159 3.14159
- joint LShoulderPitch: parent trunk_link -> torso_link
- joint RAnkleRoll: origin xyz=0 0.0275 0 rpy=-1.5707963 0 0 -> xyz=0 0 0 rpy=-1.5707963 0 0
- joint RHipPitch: origin xyz=0 0 -0.025 rpy=1.5707963 0 -1.5707963 -> xyz=0 0 0 rpy=1.5707963 0 -1.5707963
- joint RHipRoll: origin xyz=-0.025 0 0.038444 rpy=-1.5707963 0 1.5707963 -> xyz=0 0 0.038444 rpy=-1.5707963 0 1.5707963
- joint RHipYaw: origin xyz=-0.022 -0.057775 -0.160593 rpy=0 3.14159 3.14159 -> xyz=0 -0.057775 0 rpy=0 3.14159 3.14159
- joint RShoulderPitch: parent trunk_link -> torso_link
- joint j_imu: parent trunk_link -> torso_link

File: minibot_description/urdf/minibot.urdf.xacro (robot description, xacro)
@@ -7,11 +7,14 @@
 <xacro:property name="f" value="0" /> <!-- friction -->
 <xacro:property name="pos_or_eff" value="1" /> <!-- position (0) or effort(1) joint interfaces -->
-<link name="base_link"/>
-  <joint name="base_link_to_body" type="fixed">
+  <!--
+    <link name="base_link"/>
+    <joint name="base_link_to_body" type="fixed">
     <parent link="base_link"/>
     <child link="trunk_link"/>
-    <origin xyz="0 0 0.545" rpy="0 0 0" />
-  </joint>
+    <origin xyz="0 0 0.384407" rpy="0 0 0" />
+  </joint>-->
   <link name="trunk_link">
+  </link>
+  <link name="torso_link">
     <inertial>
       <origin xyz="-0.025019 0.000832 -0.054364" rpy=" 1.5707963268 0 1.5707963268"/>
@@ -265,5 +268,5 @@
     </inertial>
     <visual>
-      <origin xyz="0 0 -0.025" rpy="0 3.14 0" />
+      <origin xyz="0 0 0" rpy="0 3.14 0" />
       <geometry>
         <!--box size="0.001 0.001 0.001"/-->
@@ -275,5 +278,5 @@
     </visual>
     <collision>
-      <origin xyz="0 0 -0.025" rpy="0 3.14 0" />
+      <origin xyz="0 0 0" rpy="0 3.14 0" />
       <geometry>
         <mesh filename="package://minibot_description/meshes/hip_roll_coll.dae"  scale="1 1 1"/>
@@ -364,5 +367,5 @@
     </inertial>
     <visual>
-      <origin xyz="0 0 -0.025" rpy="0 0 -1.5707963268" />
+      <origin xyz="0 0 0" rpy="0 0 -1.5707963268" />
       <geometry>
         <!--box size="0.008 0.066 0.104"/-->
@@ -374,5 +377,5 @@
     </visual>
     <collision>
-      <origin xyz="0 0 -0.025" rpy="0 0 -1.5707963268" />
+      <origin xyz="0 0 0" rpy="0 0 -1.5707963268" />
       <geometry>
         <mesh filename="package://minibot_description/meshes/foot_coll.dae"  scale="1 1 1"/>
@@ -413,5 +416,5 @@
     </inertial>
     <visual>
-      <origin xyz="0 0 -0.025" rpy="0 3.14 0" />
+      <origin xyz="0 0 0" rpy="0 3.14 0" />
       <geometry>
         <!--box size="0.001 0.001 0.001"/-->
@@ -423,5 +426,5 @@
     </visual>
     <collision>
-      <origin xyz="0 0 -0.025" rpy="0 3.14 0" />
+      <origin xyz="0 0 0" rpy="0 3.14 0" />
       <geometry>
         <mesh filename="package://minibot_description/meshes/hip_roll_coll.dae"  scale="1 1 1"/>
@@ -512,5 +515,5 @@
     </inertial>
     <visual>
-      <origin xyz="0 0 -0.025" rpy="0 0 1.5707963268" />
+      <origin xyz="0 0 0" rpy="0 0 1.5707963268" />
       <geometry>
         <!--box size="0.008 0.066 0.104"/-->
@@ -522,5 +525,5 @@
     </visual>
     <collision>
-      <origin xyz="0 0 -0.025" rpy="0 0 1.5707963268" />
+      <origin xyz="0 0 0" rpy="0 0 1.5707963268" />
       <geometry>
         <mesh filename="package://minibot_description/meshes/foot_coll.dae"  scale="1 1 1"/>
@@ -538,7 +541,13 @@
   </link>
   <joint name="j_imu" type="fixed">
-  <parent link="trunk_link"/>
+  <parent link="torso_link"/>
   <child link="L_IMU"/>
   <origin xyz="-0.03 0 -0.05" rpy="0 0 0" />
+  <axis xyz="0 0 1" />
+  </joint>
+  <joint name="torso" type="fixed">
+  <parent link="trunk_link"/>
+  <child link="torso_link"/>
+  <origin xyz="0.022 0 0.160593" rpy="0 0 0" />
   <axis xyz="0 0 1" />
   </joint>
@@ -557,5 +566,5 @@
   <dynamics damping="${d}" friction="0.0"/> </joint>
   <joint name="HeadPan" type="revolute">
-    <parent link="trunk_link"/>
+    <parent link="torso_link"/>
     <child link="L_HEAD_PAN"/>
     <origin xyz="0 0 0.050593" rpy="0 0 1.5707963" />
@@ -564,5 +573,5 @@
   <dynamics damping="${d}" friction="0.0"/> </joint>
   <joint name="LShoulderPitch" type="revolute">
-    <parent link="trunk_link"/>
+    <parent link="torso_link"/>
     <child link="L_SHOULDER_PITCH_L"/>
     <origin xyz="0 0.08134 0" rpy="0 -1.5707963 -1.5707963" />
@@ -590,5 +599,5 @@
   </joint>
   <joint name="RShoulderPitch" type="revolute">
-    <parent link="trunk_link"/>
+    <parent link="torso_link"/>
     <child link="L_SHOULDER_PITCH_R"/>
     <origin xyz="0 -0.08134 0" rpy="0 1.5707963 -1.5707963" />
@@ -618,5 +627,5 @@
     <parent link="trunk_link"/>
     <child link="L_HIP_YAW_L"/>
-    <origin xyz="-0.022 0.057775 -0.160593" rpy="0 3.14159 3.14159" />
+    <origin xyz="0 0.057775 0" rpy="0 3.14159 3.14159" />
     <axis xyz="0 0 1" />
     <limit effort="${tofa*2.5}" velocity="5.6548668" lower="-0.9250245035547" upper="0.9250245035547" />
@@ -625,5 +634,5 @@
     <parent link="L_HIP_YAW_L"/>
     <child link="L_HIP_ROLL_L"/>
-    <origin xyz="-0.025 0 0.038444" rpy="-1.5707963 0 1.5707963" />
+    <origin xyz="0 0 0.038444" rpy="-1.5707963 0 1.5707963" />
     <axis xyz="0 0 1" />
     <limit effort="${tofa*6.0}" velocity="6.597344565" lower="-1.0122909661542001" upper="0.7853981633955001" />
@@ -632,5 +641,5 @@
     <parent link="L_HIP_ROLL_L"/>
     <child link="L_HIP_PITCH_L"/>
-    <origin xyz="0 0 -0.025" rpy="1.5707963 0 1.5707963" />
+    <origin xyz="0 0 0" rpy="1.5707963 0 1.5707963" />
     <axis xyz="0 0 1" />
     <limit effort="${tofa*8.4}" velocity="4.712388975" lower="-0.48869219055720003" upper="1.919862177189" />
@@ -653,5 +662,5 @@
     <parent link="L_ANKLE_PITCH_L"/>
     <child link="L_ANKLE_ROLL_L"/>
-    <origin xyz="0 0.0275 0" rpy="-1.5707963 0 0" />
+    <origin xyz="0 0 0" rpy="-1.5707963 0 0" />
     <axis xyz="0 0 1" />
     <limit effort="${tofa*6.0}" velocity="6.597344565" lower="-1.4660765716716" upper="1.4660765716716" />
@@ -670,5 +679,5 @@
     <parent link="trunk_link"/>
     <child link="L_HIP_YAW_R"/>
-    <origin xyz="-0.022 -0.057775 -0.160593" rpy="0 3.14159 3.14159" />
+    <origin xyz="0 -0.057775 0" rpy="0 3.14159 3.14159" />
     <axis xyz="0 0 1" />
     <limit effort="${tofa*2.5}" velocity="5.6548668" lower="-0.9250245035547" upper="0.9250245035547" />
@@ -677,5 +686,5 @@
     <parent link="L_HIP_YAW_R"/>
     <child link="L_HIP_ROLL_R"/>
-    <origin xyz="-0.025 0 0.038444" rpy="-1.5707963 0 1.5707963" />
+    <origin xyz="0 0 0.038444" rpy="-1.5707963 0 1.5707963" />
     <axis xyz="0 0 1" />
     <limit effort="${tofa*6.0}" velocity="6.597344565" lower="-1.0122909661542001" upper="0.7853981633955001" />
@@ -684,5 +693,5 @@
     <parent link="L_HIP_ROLL_R"/>
     <child link="L_HIP_PITCH_R"/>
-    <origin xyz="0 0 -0.025" rpy="1.5707963 0 -1.5707963" />
+    <origin xyz="0 0 0" rpy="1.5707963 0 -1.5707963" />
     <axis xyz="0 0 1" />
     <limit effort="${tofa*8.4}" velocity="4.712388975" lower="-1.919862177189" upper="0.48869219055720003" />
@@ -705,5 +714,5 @@
     <parent link="L_ANKLE_PITCH_R"/>
     <child link="L_ANKLE_ROLL_R"/>
-    <origin xyz="0 0.0275 0" rpy="-1.5707963 0 0" />
+    <origin xyz="0 0 0" rpy="-1.5707963 0 0" />
     <axis xyz="0 0 1" />
     <limit effort="${tofa*6.0}" velocity="6.597344565" lower="-1.4660765716716" upper="1.4660765716716" />

File: minibot_description/urdf/minibot_renamed.urdf (robot description, URDF)
Before this commit: robot Minibot, 30 links, 29 joints
Joints:
- joint right_knee: limit lower=0 upper=2.268928027587 effort=8.4 velocity=4.712388975 -> lower=-3.14 upper=3.14 effort=8.4 velocity=4.712388975

File: minibot_description/urdf/minibot_renamed.urdf.xacro (robot description, xacro)
@@ -642,5 +642,5 @@
     <axis xyz="0 0 -1" />
     <!--<limit effort="${tofa*8.4}" velocity="4.712388975" lower="-2.268928027587" upper="0" />-->
-    -<limit effort="${tofa*8.4}" velocity="4.712388975" lower="-3.14" upper="3.14" />
+    <limit effort="${tofa*8.4}" velocity="4.712388975" lower="-3.14" upper="3.14" />
   <dynamics damping="${d}" friction="0.0"/> </joint>
   <joint name="left_ankle_pitch" type="revolute">
@@ -694,5 +694,6 @@
     <origin xyz="0.150 0 0" rpy="0 0 0" />
     <axis xyz="0 0 1" />
-    <limit effort="${tofa*8.4}" velocity="4.712388975" lower="0" upper="2.268928027587" />
+    <!--<limit effort="${tofa*8.4}" velocity="4.712388975" lower="0" upper="2.268928027587" />-->
+    <limit effort="${tofa*8.4}" velocity="4.712388975" lower="-3.14" upper="3.14" />
   <dynamics damping="${d}" friction="0.0"/> </joint>
   <joint name="right_ankle_pitch" type="revolute">

Commit message: stabilizing simulation

File: minibot_description/urdf/minibot.urdf (robot description, URDF)
Before this commit: robot Minibot, 30 links, 29 joints
Links:
- link L_HEAD_PAN: mass 0.001 -> 0.1
- link L_HEAD_TILT: mass 0.001 -> 0.1

File: minibot_description/urdf/minibot.urdf.xacro (robot description, xacro)
@@ -4,5 +4,5 @@
 <xacro:property name="infa" value="1" /> <!--inertia factor-->
 <xacro:property name="insu" value="0" /> <!--inertia summand-->
-<xacro:property name="d" value="0" /> <!-- damping -->
+<xacro:property name="d" value="0.000001" /> <!-- damping -->
 <xacro:property name="f" value="0" /> <!-- friction -->
 <xacro:property name="pos_or_eff" value="1" /> <!-- position (0) or effort(1) joint interfaces -->
@@ -43,9 +43,9 @@
     <inertial>
       <origin xyz="0.000002 -0.001022 0.008994"/>
-            <mass value="0.001"/>
-      <inertia ixx="0"  ixy="0"  ixz="0" iyy="0" iyz="0" izz="0" />
+            <mass value="0.1"/>
+      <!--<inertia ixx="0"  ixy="0"  ixz="0" iyy="0" iyz="0" izz="0" />-->
       <!--<mass value="0.012"/>-->
       <!--<inertia ixx="0.000001769"  ixy="0.0"  ixz="0.0" iyy="0.000004625" iyz="-0.000000082" izz="0.000005125" />-->
-      <!--<inertia ixx="${insu*0.1+infa*0.000001769}"  ixy="0.0"  ixz="0" iyy="${insu*0.1+infa*0.000004625}" iyz="0.0" izz="${insu*0.1+infa*0.000005125}" />-->
+      <inertia ixx="${insu*0.1+infa*0.000001769}"  ixy="0.0"  ixz="0" iyy="${insu*0.1+infa*0.000004625}" iyz="0.0" izz="${insu*0.1+infa*0.000005125}" />
       <!--<inertia ixx="0.001"  ixy="0.001"  ixz="0.001" iyy="0.001" iyz="0.001" izz="0.001" />-->
     </inertial>
@@ -69,8 +69,8 @@
     <inertial>
       <origin xyz="-0.000223 -0.028433 0.0" rpy="0 1.5707963268 0"/>
-      <mass value="0.001"/>
-      <inertia ixx="0"  ixy="0"  ixz="0" iyy="0" iyz="0" izz="0" />
-      <!--<mass value="0.139"/>
-      <inertia ixx="${insu*0.1+infa*0.000097954}"  ixy="0"  ixz="0" iyy="${insu*0.1+infa*0.000025415}" iyz="0" izz="${insu*0.1+infa*0.000107764}" /> -->
+      <mass value="0.1"/>
+      <!--<inertia ixx="0"  ixy="0"  ixz="0" iyy="0" iyz="0" izz="0" />-->
+      <!--<mass value="0.139"/>-->
+      <inertia ixx="${insu*0.1+infa*0.000097954}"  ixy="0"  ixz="0" iyy="${insu*0.1+infa*0.000025415}" iyz="0" izz="${insu*0.1+infa*0.000107764}" />
       <!--<inertia ixx="0.001"  ixy="0.001"  ixz="0.001" iyy="0.001" iyz="0.001" izz="0.001" />-->
     </inertial>
@@ -1178,8 +1178,8 @@
 <gazebo reference="L_ANKLE_ROLL_L">
     <material>Gazebo/Grey</material>
-      <kp>1000000.0</kp>
+      <kp>100000.0</kp>
       <kd>100.0</kd>
-      <mu1>1.0</mu1>
-      <mu2>1.0</mu2>
+      <mu1>50.0</mu1>
+      <mu2>50.0</mu2>
       <fdir1>1 0 0</fdir1>
       <maxVel>1.0</maxVel>
