Commit message: changed trunk link to base link

File: minibot_description/urdf/minibot.urdf (robot description, URDF)
Before this commit: robot Minibot, 30 links, 29 joints
Links:
- removed link trunk_link
- added link base_link
Joints:
- joint LHipYaw: parent trunk_link -> base_link
- joint RHipYaw: parent trunk_link -> base_link
- joint torso: parent trunk_link -> base_link

File: minibot_description/urdf/minibot.urdf.xacro (robot description, xacro)
@@ -11,8 +11,8 @@
     <joint name="base_link_to_body" type="fixed">
     <parent link="base_link"/>
-    <child link="trunk_link"/>
+    <child link="base_link"/>
     <origin xyz="0 0 0.384407" rpy="0 0 0" />
   </joint>-->
-  <link name="trunk_link">
+  <link name="base_link">
   </link>
   <link name="torso_link">
@@ -547,5 +547,5 @@
   </joint>
   <joint name="torso" type="fixed">
-  <parent link="trunk_link"/>
+  <parent link="base_link"/>
   <child link="torso_link"/>
   <origin xyz="0.022 0 0.160593" rpy="0 0 0" />
@@ -625,5 +625,5 @@
   </joint>
   <joint name="LHipYaw" type="revolute">
-    <parent link="trunk_link"/>
+    <parent link="base_link"/>
     <child link="L_HIP_YAW_L"/>
     <origin xyz="0 0.057775 0" rpy="0 3.14159 3.14159" />
@@ -677,5 +677,5 @@
   </joint>
   <joint name="RHipYaw" type="revolute">
-    <parent link="trunk_link"/>
+    <parent link="base_link"/>
     <child link="L_HIP_YAW_R"/>
     <origin xyz="0 -0.057775 0" rpy="0 3.14159 3.14159" />
@@ -1128,5 +1128,5 @@
     </actuator>
   </transmission>
-<gazebo reference="trunk_link">
+<gazebo reference="base_link">
     <material>Gazebo/Grey</material>
   </gazebo>
