Commit message: renamed minibot urdf to follow REP-120

File: minibot_description/urdf/minibot.urdf (robot description, URDF)
Before this commit: robot Minibot, 30 links, 29 joints
Links:
- removed link L_ANKLE_PITCH_L
- removed link L_ANKLE_PITCH_R
- removed link L_ANKLE_ROLL_L
- removed link L_ANKLE_ROLL_R
- removed link L_CAMERA
- removed link L_ELBOW_L
- removed link L_ELBOW_R
- removed link L_FOOT_FRONT_L
- removed link L_FOOT_FRONT_R
- removed link L_HEAD_PAN
- removed link L_HEAD_TILT
- removed link L_HIP_PITCH_L
- removed link L_HIP_PITCH_R
- removed link L_HIP_ROLL_L
- removed link L_HIP_ROLL_R
- removed link L_HIP_YAW_L
- removed link L_HIP_YAW_R
- removed link L_Hand_L
- removed link L_Hand_R
- removed link L_IMU
- removed link L_KNEE_L
- removed link L_KNEE_R
- removed link L_SHOULDER_PITCH_L
- removed link L_SHOULDER_PITCH_R
- removed link L_SHOULDER_ROLL_L
- removed link L_SHOULDER_ROLL_R
- removed link left_foot_sole_link
- removed link right_foot_sole_link
- removed link torso_link
- added link camera
- added link head, mass 0.1; collision mesh filename=package://minibot_description/meshes/head_upper_coll.dae scale=1 1 1; visual mesh filename=package://minibot_description/meshes/head_upper_high.stl scale=1 1 1
- added link imu
- added link l_ankle, mass 0.325; collision mesh filename=package://minibot_description/meshes/ankle_roll_coll.dae scale=1 1 1; visual mesh filename=package://minibot_description/meshes/ankle_roll_low.dae scale=1 1 1
- added link l_foot, mass 0.086; collision mesh filename=package://minibot_description/meshes/foot_coll.dae scale=1 1 1; visual mesh filename=package://minibot_description/meshes/foot_high.stl scale=1 1 1
- added link l_hip_1, mass 0.022; collision mesh filename=package://minibot_description/meshes/yaw_con_coll.dae scale=1 1 1; visual mesh filename=package://minibot_description/meshes/yaw_con_high.stl scale=1 1 1
- added link l_hip_2, mass 0.325; collision mesh filename=package://minibot_description/meshes/hip_roll_coll.dae scale=1 1 1; visual mesh filename=package://minibot_description/meshes/hip_roll_low.dae scale=1 1 1
- added link l_lower_arm, mass 0.097; collision mesh filename=package://minibot_description/meshes/lower_arm_coll.dae scale=1 1 1; visual mesh filename=package://minibot_description/meshes/lower_arm_high.stl scale=1 1 1
- added link l_lower_leg, mass 0.055; collision mesh filename=package://minibot_description/meshes/lower_leg_coll.dae scale=1 1 1; visual mesh filename=package://minibot_description/meshes/lower_leg_high.stl scale=1 1 1
- added link l_shoulder, mass 0.018; collision mesh filename=package://minibot_description/meshes/shoulder_con_coll.dae scale=1 1 1; visual mesh filename=package://minibot_description/meshes/shoulder_con_high.stl scale=1 1 1
- added link l_sole
- added link l_toe
- added link l_upper_arm, mass 0.190; collision mesh filename=package://minibot_description/meshes/upper_arm_coll.dae scale=1 1 1; visual mesh filename=package://minibot_description/meshes/upper_arm_high.dae scale=1 1 1
- added link l_upper_leg, mass 0.215; collision mesh filename=package://minibot_description/meshes/upper_leg_coll.dae scale=1 1 1; visual mesh filename=package://minibot_description/meshes/upper_leg_high.stl scale=1 1 1
- added link l_wrist
- added link neck, mass 0.1; collision mesh filename=package://minibot_description/meshes/head_lower_coll.dae scale=1 1 1; visual mesh filename=package://minibot_description/meshes/head_lower_high.stl scale=1 1 1
- added link r_ankle, mass 0.325; collision mesh filename=package://minibot_description/meshes/ankle_roll_coll.dae scale=1 1 1; visual mesh filename=package://minibot_description/meshes/ankle_roll_low.dae scale=1 1 1
- added link r_foot, mass 0.086; collision mesh filename=package://minibot_description/meshes/foot_coll.dae scale=1 1 1; visual mesh filename=package://minibot_description/meshes/foot_high.stl scale=1 1 1
- added link r_hip_1, mass 0.022; collision mesh filename=package://minibot_description/meshes/yaw_con_coll.dae scale=1 1 1; visual mesh filename=package://minibot_description/meshes/yaw_con_high.stl scale=1 1 1
- added link r_hip_2, mass 0.325; collision mesh filename=package://minibot_description/meshes/hip_roll_coll.dae scale=1 1 1; visual mesh filename=package://minibot_description/meshes/hip_roll_low.dae scale=1 1 1
- added link r_lower_arm, mass 0.097; collision mesh filename=package://minibot_description/meshes/lower_arm_coll.dae scale=1 1 1; visual mesh filename=package://minibot_description/meshes/lower_arm_high.stl scale=1 1 1
- added link r_lower_leg, mass 0.055; collision mesh filename=package://minibot_description/meshes/lower_leg_coll.dae scale=1 1 1; visual mesh filename=package://minibot_description/meshes/lower_leg_high.stl scale=1 1 1
- added link r_shoulder, mass 0.018; collision mesh filename=package://minibot_description/meshes/shoulder_con_coll.dae scale=1 1 1; visual mesh filename=package://minibot_description/meshes/shoulder_con_high.stl scale=1 1 1
- added link r_sole
- added link r_toe
- added link r_upper_arm, mass 0.190; collision mesh filename=package://minibot_description/meshes/upper_arm_coll.dae scale=1 1 1; visual mesh filename=package://minibot_description/meshes/upper_arm_high.dae scale=1 1 1
- added link r_upper_leg, mass 0.215; collision mesh filename=package://minibot_description/meshes/upper_leg_coll.dae scale=1 1 1; visual mesh filename=package://minibot_description/meshes/upper_leg_high.stl scale=1 1 1
- added link r_wrist
- added link torso, mass 1.423; collision mesh filename=package://minibot_description/meshes/torso_coll.dae scale=1 1 1; visual mesh filename=package://minibot_description/meshes/torso_low.dae scale=1 1 1
Joints:
- removed joint j_LFootBottom
- removed joint j_LFootFront
- removed joint j_LHand
- removed joint j_RFootBottom
- removed joint j_RFootFront
- removed joint j_RHand
- removed joint j_camboard
- removed joint j_imu
- removed joint torso
- added joint base_to_torso: type fixed, parent base_link, child torso, origin xyz=0.022 0 0.160593 rpy=0 0 0, axis 0 0 1
- added joint head_to_camera: type fixed, parent head, child camera, origin xyz=0 -0.055 0  rpy=-1.5707963 0 3.14159, axis 0 0 1
- added joint l_elbow_to_hand: type fixed, parent l_lower_arm, child l_wrist, origin xyz=-0.1573 0 0 rpy=0 0 3.14159
- added joint l_foot_to_sole: type fixed, parent l_foot, child l_sole, origin xyz=-0.040444 0 0 rpy=3.14159 -1.5707963 0
- added joint l_sole_to_toe: type fixed, parent l_sole, child l_toe, origin xyz=0.0849 0 0 
- added joint r_elbow_to_hand: type fixed, parent r_lower_arm, child r_wrist, origin xyz=0.1573 0 0
- added joint r_foot_to_sole: type fixed, parent r_foot, child r_sole, origin xyz=0.040444 0 0 rpy=0 -1.5707963 0
- added joint r_sole_to_toe: type fixed, parent r_sole, child r_toe, origin xyz=0.0849 0 0 
- added joint torso_to_imu: type fixed, parent torso, child imu, origin xyz=-0.03 0 -0.05 rpy=0 0 0, axis 0 0 1
- joint HeadPan: child L_HEAD_PAN -> neck; parent torso_link -> torso
- joint HeadTilt: child L_HEAD_TILT -> head; parent L_HEAD_PAN -> neck
- joint LAnklePitch: child L_ANKLE_PITCH_L -> l_ankle; parent L_KNEE_L -> l_lower_leg
- joint LAnkleRoll: child L_ANKLE_ROLL_L -> l_foot; parent L_ANKLE_PITCH_L -> l_ankle
- joint LElbow: child L_ELBOW_L -> l_lower_arm; parent L_SHOULDER_ROLL_L -> l_upper_arm
- joint LHipPitch: child L_HIP_PITCH_L -> l_upper_leg; parent L_HIP_ROLL_L -> l_hip_2
- joint LHipRoll: child L_HIP_ROLL_L -> l_hip_2; parent L_HIP_YAW_L -> l_hip_1
- joint LHipYaw: child L_HIP_YAW_L -> l_hip_1
- joint LKnee: child L_KNEE_L -> l_lower_leg; parent L_HIP_PITCH_L -> l_upper_leg
- joint LShoulderPitch: child L_SHOULDER_PITCH_L -> l_shoulder; parent torso_link -> torso
- joint LShoulderRoll: child L_SHOULDER_ROLL_L -> l_upper_arm; parent L_SHOULDER_PITCH_L -> l_shoulder
- joint RAnklePitch: child L_ANKLE_PITCH_R -> r_ankle; parent L_KNEE_R -> r_lower_leg
- joint RAnkleRoll: child L_ANKLE_ROLL_R -> r_foot; parent L_ANKLE_PITCH_R -> r_ankle
- joint RElbow: child L_ELBOW_R -> r_lower_arm; parent L_SHOULDER_ROLL_R -> r_upper_arm
- joint RHipPitch: child L_HIP_PITCH_R -> r_upper_leg; parent L_HIP_ROLL_R -> r_hip_2
- joint RHipRoll: child L_HIP_ROLL_R -> r_hip_2; parent L_HIP_YAW_R -> r_hip_1
- joint RHipYaw: child L_HIP_YAW_R -> r_hip_1
- joint RKnee: child L_KNEE_R -> r_lower_leg; parent L_HIP_PITCH_R -> r_upper_leg
- joint RShoulderPitch: child L_SHOULDER_PITCH_R -> r_shoulder; parent torso_link -> torso
- joint RShoulderRoll: child L_SHOULDER_ROLL_R -> r_upper_arm; parent L_SHOULDER_PITCH_R -> r_shoulder

File: minibot_description/urdf/minibot.urdf.xacro (robot description, xacro)
@@ -7,14 +7,7 @@
 <xacro:property name="f" value="0" /> <!-- friction -->
 <xacro:property name="pos_or_eff" value="1" /> <!-- position (0) or effort(1) joint interfaces -->
-  <!--
-    <link name="base_link"/>
-    <joint name="base_link_to_body" type="fixed">
-    <parent link="base_link"/>
-    <child link="base_link"/>
-    <origin xyz="0 0 0.384407" rpy="0 0 0" />
-  </joint>-->
   <link name="base_link">
   </link>
-  <link name="torso_link">
+  <link name="torso">
     <inertial>
       <origin xyz="-0.025019 0.000832 -0.054364" rpy=" 1.5707963268 0 1.5707963268"/>
@@ -40,5 +33,5 @@
     </collision> -->
   </link>
-  <link name="L_HEAD_PAN">
+  <link name="neck">
     <inertial>
       <origin xyz="0.000002 -0.001022 0.008994"/>
@@ -66,5 +59,5 @@
     </collision>
   </link>
-  <link name="L_HEAD_TILT">
+  <link name="head">
     <inertial>
       <origin xyz="-0.000223 -0.028433 0.0" rpy="0 1.5707963268 0"/>
@@ -91,5 +84,5 @@
     </collision>
   </link>
-  <link name="L_SHOULDER_PITCH_L">
+  <link name="l_shoulder">
     <inertial>
       <origin xyz="0.0 0.0 0.0087"/>
@@ -115,5 +108,5 @@
     </collision>
   </link>
-  <link name="L_SHOULDER_ROLL_L" >
+  <link name="l_upper_arm" >
     <inertial>
       <origin xyz="-0.071053 0.000432 0.000046"/>
@@ -139,5 +132,5 @@
     </collision>
   </link>
-  <link name="L_ELBOW_L" >
+  <link name="l_lower_arm" >
     <inertial>
       <origin xyz="-0.108 0.0 0.0" rpy="0 0 -3.141"/>
@@ -162,5 +155,5 @@
     </collision>
   </link>
-  <link name="L_SHOULDER_PITCH_R" >
+  <link name="r_shoulder" >
     <inertial>
       <origin xyz="0.0 0.0 0.0087"/>
@@ -186,5 +179,5 @@
     </collision>
   </link>
-  <link name="L_SHOULDER_ROLL_R" >
+  <link name="r_upper_arm" >
     <inertial>
       <origin xyz="-0.071053 0.000432 0.000046"/>
@@ -211,5 +204,5 @@
     </collision>
   </link>
-  <link name="L_ELBOW_R" >
+  <link name="r_lower_arm" >
     <inertial>
       <!--<origin xyz="0.108 0.0 0.0" rpy="0 1.5707963268 1.5707963268"/>-->
@@ -235,5 +228,5 @@
     </collision>
   </link>
-  <link name="L_HIP_YAW_L" >
+  <link name="l_hip_1" >
     <inertial>
       <origin xyz="0.0 0.0 0.011" rpy="1.5707963268 0 1.5707963268"/>
@@ -259,5 +252,5 @@
     </collision>
   </link>
-  <link name="L_HIP_ROLL_L" >
+  <link name="l_hip_2" >
     <inertial>
       <origin xyz="-0.00057 -0.013721 0.02013 "/>
@@ -284,5 +277,5 @@
     </collision>
   </link>
-  <link name="L_HIP_PITCH_L" >
+  <link name="l_upper_leg" >
     <inertial>
       <origin xyz="-0.12799 -0.000699 0.000454" rpy="0 1.5707963268 1.5707963268"/>
@@ -309,5 +302,5 @@
     </collision>
   </link>
-  <link name="L_KNEE_L" >
+  <link name="l_lower_leg" >
     <inertial>
       <origin xyz="-0.072079 -0.00295 0.0" rpy="0 1.5707963268 1.5707963268"/>
@@ -334,5 +327,5 @@
     </collision>
   </link>
-  <link name="L_ANKLE_PITCH_L" >
+  <link name="l_ankle" >
     <inertial>
       <origin xyz="0.014045 -0.020134 -0.000053" rpy="1.5707963268 1.5707963268 0"/>
@@ -359,5 +352,5 @@
     </collision>
   </link>
-  <link name="L_ANKLE_ROLL_L" >
+  <link name="l_foot" >
     <inertial>
       <origin xyz="-0.0364 0.0003 0.002423" rpy="0 0 1.5707963268"/>
@@ -383,5 +376,5 @@
     </collision>
   </link>
-  <link name="L_HIP_YAW_R" >
+  <link name="r_hip_1" >
     <inertial>
       <origin xyz="0.0 0.0 0.011" rpy="1.5707963268 0 1.5707963268"/>
@@ -407,5 +400,5 @@
     </collision>
   </link>
-  <link name="L_HIP_ROLL_R" >
+  <link name="r_hip_2" >
     <inertial>
       <origin xyz="-0.00057 -0.013721 0.02013 "/>
@@ -432,5 +425,5 @@
     </collision>
   </link>
-  <link name="L_HIP_PITCH_R" >
+  <link name="r_upper_leg" >
     <inertial>
       <origin xyz="0.12799 -0.000699 0.000454" rpy="0 1.5707963268 1.5707963268"/>
@@ -457,5 +450,5 @@
     </collision>
   </link>
-  <link name="L_KNEE_R" >
+  <link name="r_lower_leg" >
     <inertial>
       <origin xyz="0.072079 -0.00295 0.0" rpy="0 1.5707963268 1.5707963268"/>
@@ -482,5 +475,5 @@
     </collision>
   </link>
-  <link name="L_ANKLE_PITCH_R" >
+  <link name="r_ankle" >
     <inertial>
       <origin xyz="-0.014045 -0.020134 -0.000053" rpy="1.5707963268 1.5707963268 0"/>
@@ -507,5 +500,5 @@
     </collision>
   </link>
-  <link name="L_ANKLE_ROLL_R" >
+  <link name="r_foot" >
     <inertial>
       <origin xyz="0.0364 0.0003 0.002423" rpy="0 0 1.5707963268"/>
@@ -531,34 +524,34 @@
     </collision>
   </link>
-  <link name="L_CAMERA" />
-  <link name="L_Hand_L" />
-  <link name="L_Hand_R" />
-  <link name="left_foot_sole_link" />
-  <link name="right_foot_sole_link" />
-  <link name="L_FOOT_FRONT_L" />
-  <link name="L_FOOT_FRONT_R" />
-  <link name="L_IMU">
-  </link>
-  <joint name="j_imu" type="fixed">
-  <parent link="torso_link"/>
-  <child link="L_IMU"/>
+  <link name="camera" />
+  <link name="l_wrist" />
+  <link name="r_wrist" />
+  <link name="l_sole" />
+  <link name="r_sole" />
+  <link name="l_toe" />
+  <link name="r_toe" />
+  <link name="imu">
+  </link>
+  <joint name="torso_to_imu" type="fixed">
+  <parent link="torso"/>
+  <child link="imu"/>
   <origin xyz="-0.03 0 -0.05" rpy="0 0 0" />
   <axis xyz="0 0 1" />
   </joint>
-  <joint name="torso" type="fixed">
+  <joint name="base_to_torso" type="fixed">
   <parent link="base_link"/>
-  <child link="torso_link"/>
+  <child link="torso"/>
   <origin xyz="0.022 0 0.160593" rpy="0 0 0" />
   <axis xyz="0 0 1" />
   </joint>
-  <joint name="j_camboard" type="fixed">
-  <parent link="L_HEAD_TILT"/>
-  <child link="L_CAMERA"/>
+  <joint name="head_to_camera" type="fixed">
+  <parent link="head"/>
+  <child link="camera"/>
   <origin xyz="0 -0.055 0 " rpy="-1.5707963 0 3.14159" />
   <axis xyz="0 0 1" />
   </joint>
   <joint name="HeadTilt" type="revolute">
-    <parent link="L_HEAD_PAN"/>
-    <child link="L_HEAD_TILT"/>
+    <parent link="neck"/>
+    <child link="head"/>
     <origin xyz="0 0 0.02715" rpy="-1.5707963 0 1.5707963" />
     <axis xyz="0 0 1" />
@@ -566,6 +559,6 @@
   <dynamics damping="${d}" friction="0.0"/> </joint>
   <joint name="HeadPan" type="revolute">
-    <parent link="torso_link"/>
-    <child link="L_HEAD_PAN"/>
+    <parent link="torso"/>
+    <child link="neck"/>
     <origin xyz="0 0 0.050593" rpy="0 0 1.5707963" />
     <axis xyz="0 0 1" />
@@ -573,6 +566,6 @@
   <dynamics damping="${d}" friction="0.0"/> </joint>
   <joint name="LShoulderPitch" type="revolute">
-    <parent link="torso_link"/>
-    <child link="L_SHOULDER_PITCH_L"/>
+    <parent link="torso"/>
+    <child link="l_shoulder"/>
     <origin xyz="0 0.08134 0" rpy="0 -1.5707963 -1.5707963" />
     <axis xyz="0 0 1" />
@@ -580,6 +573,6 @@
   <dynamics damping="${d}" friction="0.0"/> </joint>
   <joint name="LShoulderRoll" type="revolute">
-    <parent link="L_SHOULDER_PITCH_L"/>
-    <child link="L_SHOULDER_ROLL_L"/>
+    <parent link="l_shoulder"/>
+    <child link="l_upper_arm"/>
     <origin xyz="0 0 0.029194" rpy="-1.5707963 0.7853981633955001 0" />
     <axis xyz="0 0 -1" />
@@ -587,18 +580,18 @@
   <dynamics damping="${d}" friction="0.0"/> </joint>
   <joint name="LElbow" type="revolute">
-    <parent link="L_SHOULDER_ROLL_L"/>
-    <child link="L_ELBOW_L"/>
+    <parent link="l_upper_arm"/>
+    <child link="l_lower_arm"/>
     <origin xyz="-0.14 0 0" rpy="1.5707963 1.5707963 0" />
     <axis xyz="0 0 1" />
     <limit effort="${tofa*2.5}" velocity="5.6548668" lower="-1.1344640137935" upper="1.5707963267910001" />
   <dynamics damping="${d}" friction="0.0"/> </joint>
-  <joint name="j_LHand" type="fixed">
-   <parent link="L_ELBOW_L"/>
-   <child link="L_Hand_L" />
+  <joint name="l_elbow_to_hand" type="fixed">
+   <parent link="l_lower_arm"/>
+   <child link="l_wrist" />
    <origin xyz="-0.1573 0 0" rpy="0 0 3.14159"/>
   </joint>
   <joint name="RShoulderPitch" type="revolute">
-    <parent link="torso_link"/>
-    <child link="L_SHOULDER_PITCH_R"/>
+    <parent link="torso"/>
+    <child link="r_shoulder"/>
     <origin xyz="0 -0.08134 0" rpy="0 1.5707963 -1.5707963" />
     <axis xyz="0 0 1" />
@@ -606,6 +599,6 @@
   <dynamics damping="${d}" friction="0.0"/> </joint>
   <joint name="RShoulderRoll" type="revolute">
-    <parent link="L_SHOULDER_PITCH_R"/>
-    <child link="L_SHOULDER_ROLL_R"/>
+    <parent link="r_shoulder"/>
+    <child link="r_upper_arm"/>
     <origin xyz="0 0 0.029194" rpy="-1.5707963 2.356194463 0" />
     <axis xyz="0 0 -1" />
@@ -613,18 +606,18 @@
   <dynamics damping="${d}" friction="0.0"/> </joint>
   <joint name="RElbow" type="revolute">
-    <parent link="L_SHOULDER_ROLL_R"/>
-    <child link="L_ELBOW_R"/>
+    <parent link="r_upper_arm"/>
+    <child link="r_lower_arm"/>
     <origin xyz="-0.14 0 0" rpy="-1.5707963 -1.5707963 0" />
     <axis xyz="0 0 1" />
     <limit effort="${tofa*2.5}" velocity="5.6548668" lower="-1.635" upper="1.5707963267910001" />
   <dynamics damping="${d}" friction="0.0"/> </joint>
-  <joint name="j_RHand" type="fixed">
-   <parent link="L_ELBOW_R"/>
-   <child link="L_Hand_R" />
+  <joint name="r_elbow_to_hand" type="fixed">
+   <parent link="r_lower_arm"/>
+   <child link="r_wrist" />
    <origin xyz="0.1573 0 0"/>
   </joint>
   <joint name="LHipYaw" type="revolute">
     <parent link="base_link"/>
-    <child link="L_HIP_YAW_L"/>
+    <child link="l_hip_1"/>
     <origin xyz="0 0.057775 0" rpy="0 3.14159 3.14159" />
     <axis xyz="0 0 1" />
@@ -632,6 +625,6 @@
   <dynamics damping="${d}" friction="0.0"/> </joint>
   <joint name="LHipRoll" type="revolute">
-    <parent link="L_HIP_YAW_L"/>
-    <child link="L_HIP_ROLL_L"/>
+    <parent link="l_hip_1"/>
+    <child link="l_hip_2"/>
     <origin xyz="0 0 0.038444" rpy="-1.5707963 0 1.5707963" />
     <axis xyz="0 0 1" />
@@ -639,6 +632,6 @@
   <dynamics damping="${d}" friction="0.0"/> </joint>
   <joint name="LHipPitch" type="revolute">
-    <parent link="L_HIP_ROLL_L"/>
-    <child link="L_HIP_PITCH_L"/>
+    <parent link="l_hip_2"/>
+    <child link="l_upper_leg"/>
     <origin xyz="0 0 0" rpy="1.5707963 0 1.5707963" />
     <axis xyz="0 0 1" />
@@ -646,6 +639,6 @@
   <dynamics damping="${d}" friction="0.0"/> </joint>
   <joint name="LKnee" type="revolute">
-    <parent link="L_HIP_PITCH_L"/>
-    <child link="L_KNEE_L"/>
+    <parent link="l_upper_leg"/>
+    <child link="l_lower_leg"/>
     <origin xyz="-0.150 0 0" rpy="0 0 0" />
     <axis xyz="0 0 1" />
@@ -653,6 +646,6 @@
   <dynamics damping="${d}" friction="0.0"/> </joint>
   <joint name="LAnklePitch" type="revolute">
-    <parent link="L_KNEE_L"/>
-    <child link="L_ANKLE_PITCH_L"/>
+    <parent link="l_lower_leg"/>
+    <child link="l_ankle"/>
     <origin xyz="-0.150 0 0" rpy="3.14159 0 0" />
     <axis xyz="0 0 1" />
@@ -660,23 +653,23 @@
   <dynamics damping="${d}" friction="0.0"/> </joint>
   <joint name="LAnkleRoll" type="revolute">
-    <parent link="L_ANKLE_PITCH_L"/>
-    <child link="L_ANKLE_ROLL_L"/>
+    <parent link="l_ankle"/>
+    <child link="l_foot"/>
     <origin xyz="0 0 0" rpy="-1.5707963 0 0" />
     <axis xyz="0 0 1" />
     <limit effort="${tofa*6.0}" velocity="6.597344565" lower="-1.4660765716716" upper="1.4660765716716" />
   <dynamics damping="${d}" friction="0.0"/> </joint>
-  <joint name="j_LFootBottom" type="fixed">
-   <parent link="L_ANKLE_ROLL_L"/>
-   <child link="left_foot_sole_link" />
+  <joint name="l_foot_to_sole" type="fixed">
+   <parent link="l_foot"/>
+   <child link="l_sole" />
    <origin xyz="-0.040444 0 0" rpy="3.14159 -1.5707963 0"/>
   </joint>
-  <joint name="j_LFootFront" type="fixed">
-   <parent link="left_foot_sole_link"/>
-   <child link="L_FOOT_FRONT_L" />
+  <joint name="l_sole_to_toe" type="fixed">
+   <parent link="l_sole"/>
+   <child link="l_toe" />
    <origin xyz="0.0849 0 0 "/>
   </joint>
   <joint name="RHipYaw" type="revolute">
     <parent link="base_link"/>
-    <child link="L_HIP_YAW_R"/>
+    <child link="r_hip_1"/>
     <origin xyz="0 -0.057775 0" rpy="0 3.14159 3.14159" />
     <axis xyz="0 0 1" />
@@ -684,6 +677,6 @@
   <dynamics damping="${d}" friction="0.0"/> </joint>
   <joint name="RHipRoll" type="revolute">
-    <parent link="L_HIP_YAW_R"/>
-    <child link="L_HIP_ROLL_R"/>
+    <parent link="r_hip_1"/>
+    <child link="r_hip_2"/>
     <origin xyz="0 0 0.038444" rpy="-1.5707963 0 1.5707963" />
     <axis xyz="0 0 1" />
@@ -691,6 +684,6 @@
   <dynamics damping="${d}" friction="0.0"/> </joint>
   <joint name="RHipPitch" type="revolute">
-    <parent link="L_HIP_ROLL_R"/>
-    <child link="L_HIP_PITCH_R"/>
+    <parent link="r_hip_2"/>
+    <child link="r_upper_leg"/>
     <origin xyz="0 0 0" rpy="1.5707963 0 -1.5707963" />
     <axis xyz="0 0 1" />
@@ -698,6 +691,6 @@
   <dynamics damping="${d}" friction="0.0"/> </joint>
   <joint name="RKnee" type="revolute">
-    <parent link="L_HIP_PITCH_R"/>
-    <child link="L_KNEE_R"/>
+    <parent link="r_upper_leg"/>
+    <child link="r_lower_leg"/>
     <origin xyz="0.150 0 0" rpy="0 0 0" />
     <axis xyz="0 0 1" />
@@ -705,6 +698,6 @@
   <dynamics damping="${d}" friction="0.0"/> </joint>
   <joint name="RAnklePitch" type="revolute">
-    <parent link="L_KNEE_R"/>
-    <child link="L_ANKLE_PITCH_R"/>
+    <parent link="r_lower_leg"/>
+    <child link="r_ankle"/>
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