Commit message: small xml fix

File: minibot_description/urdf/minibot.urdf.xacro (robot description, xacro)
@@ -31,5 +31,5 @@
         <mesh filename="package://minibot_description/meshes/torso_coll.dae"  scale="1 1 1"/>
       </geometry>
-    </collision> -->
+    </collision>
   </link>
   <link name="neck">

Commit message: added camera fixed frame for looking at things

File: minibot_description/urdf/minibot.urdf.xacro (robot description, xacro)
@@ -534,4 +534,6 @@
   <link name="imu">
   </link>
+  <link name="camera_fixed">
+  </link>
   <joint name="torso_to_imu" type="fixed">
   <parent link="torso"/>
@@ -544,4 +546,10 @@
   <child link="torso"/>
   <origin xyz="0.022 0 0.160593" rpy="0 0 0" />
+  <axis xyz="0 0 1" />
+  </joint>
+  <joint name="torso_to_camera_fixed" type="fixed">
+  <parent link="torso"/>
+  <child link="camera_fixed"/>
+  <origin xyz="0.0 0 0.10" rpy="0 0 0" />
   <axis xyz="0 0 1" />
   </joint>

Commit message: Correct position of camera_fixed frame

File: minibot_description/urdf/minibot.urdf.xacro (robot description, xacro)
@@ -551,5 +551,5 @@
   <parent link="torso"/>
   <child link="camera_fixed"/>
-  <origin xyz="0.0 0 0.10" rpy="0 0 0" />
+  <origin xyz="0.0 0 0.133" rpy="0 0 0" />
   <axis xyz="0 0 1" />
   </joint>
